File: carte-asser-1A-2016-2017/carte-asser-1A-2016-2017.sch (KiCad schematic (older format))
At the start: 11 parts

Commit message: Fin PCB
Parts:
- removed D? (x7): D_Small, symbol D_Small
- added P?: CONN_01X02, symbol CONN_01X02
- added R?: 1k, symbol R
- gave numbers to parts that had none: 4
Connections:
- net +8V: now also P1.1 (P1), P1.2 (P2), P1.3 (P3), P1.4 (P4), P1.5 (P5), P1.6 (P6), P1.7 (P7)
- net command_part/RX-Pi: now also P3.1 (P1)
- net command_part/RX-cervo: now also P4.1 (P1)
- net command_part/Rx-balise: now also P2.1 (P1)
- net command_part/TX-Pi: now also P3.2 (P2)
- net command_part/TX-cervo: now also P4.2 (P2)
- net command_part/Tx-balise: now also P2.2 (P2)
- new net: P?.1 (P1), R?.1
- new net GND: R?.2
- new net command_part/led_fusée: P?.2 (P2)

Commit message: PCB
Parts:
- removed P1: CONN_01X07, symbol CONN_01X07
- removed P2: CONN_01X03, symbol CONN_01X03
- removed P4: CONN_01X02, symbol CONN_01X02
- added P2: Balise, Pin_Headers:Pin_Header_Straight_1x04_Pitch2.54mm, symbol CONN_01X04
- P1: renamed from P?; value CONN_01X02 -> led-fusée; footprint (none) -> Pin_Headers:Pin_Header_Straight_1x02_Pitch2.54mm
- P3: value CONN_01X02 -> uart-pi; footprint (none) -> Pin_Headers:Pin_Header_Straight_1x02_Pitch2.54mm
- R16: renamed from R?; footprint (none) -> Discret:R4-LARGE_PADS
Connections:
- net +15V: now also P2.4 (P4)
- net GND: now also P2.1 (P1)
- net command_part/Rx-balise: now also P2.2 (P2)
- net command_part/Tx-balise: now also P2.3 (P3)
Changed lines of the file:
@@
 $Descr A2 23386 16535
 encoding utf-8
-Sheet 1 8
+Sheet 1 9
 Title ""
 Date ""
@@
 $EndSheet
 $Comp
-L CONN_01X02 P3
-U 1 1 589450AF
-P 6400 3950
-F 0 "P3" H 6400 4100 50  0000 C CNN
-F 1 "CONN_01X02" V 6500 3950 50  0000 C CNN
-F 2 "" H 6400 3950 50  0000 C CNN
-F 3 "" H 6400 3950 50  0000 C CNN
-	1    6400 3950
-	-1   0    0    1
-$EndComp
-$Comp
-L CONN_01X02 P4
-U 1 1 589C954C
-P 6400 4800
-F 0 "P4" H 6400 4950 50  0000 C CNN
-F 1 "CONN_01X02" V 6500 4800 50  0000 C CNN
-F 2 "" H 6400 4800 50  0000 C CNN
-F 3 "" H 6400 4800 50  0000 C CNN
-	1    6400 4800
-	-1   0    0    1
-$EndComp
-$Comp
-L CONN_01X03 P2
-U 1 1 589D4125
-P 5800 5850
-F 0 "P2" H 5800 6050 50  0000 C CNN
-F 1 "CONN_01X03" V 5900 5850 50  0000 C CNN
-F 2 "" H 5800 5850 50  0000 C CNN
-F 3 "" H 5800 5850 50  0000 C CNN
-	1    5800 5850
-	-1   0    0    1
-$EndComp
-$Comp
 L +15V #PWR01
 U 1 1 589D46CA
@@
 	1    0    0    -1
 $EndComp
-$Comp
-L CONN_01X07 P1
-U 1 1 589DB597
-P 4250 3800
-F 0 "P1" H 4250 4200 50  0000 C CNN
-F 1 "CONN_01X07" V 4350 3800 50  0000 C CNN
-F 2 "" H 4250 3800 50  0000 C CNN
-F 3 "" H 4250 3800 50  0000 C CNN
-	1    4250 3800
-	-1   0    0    1
-$EndComp
-$Comp
-L +8V #PWR02
-U 1 1 589DBCE6
-P 4450 2950
-F 0 "#PWR02" H 4450 2800 50  0001 C CNN
-F 1 "+8V" H 4450 3090 50  0000 C CNN
-F 2 "" H 4450 2950 50  0000 C CNN
-F 3 "" H 4450 2950 50  0000 C CNN
-	1    4450 2950
-	1    0    0    -1
-$EndComp
-Wire Wire Line
-	13300 4250 13850 4250
-Wire Wire Line
-	13300 4400 13850 4400
-Wire Wire Line
-	13300 4550 13850 4550
-Wire Wire Line
-	13850 4700 13300 4700
-Wire Wire Line
-	13300 4850 13850 4850
-Wire Wire Line
-	13850 5000 13300 5000
-Wire Wire Line
-	13850 5300 13300 5300
-Wire Wire Line
-	13300 5450 13850 5450
-Wire Wire Line
-	13300 7300 13850 7300
-Wire Wire Line
-	13850 7100 13300 7100
-Wire Wire Line
-	13300 6900 13850 6900
-Wire Wire Line
-	13850 6650 13300 6650
-Wire Wire Line
-	13300 5850 13850 5850
-Wire Wire Line
-	13300 6000 13850 6000
-Wire Wire Line
-	13850 6150 13300 6150
-Wire Wire Line
-	13300 6300 13850 6300
-Wire Wire Line
-	13850 6500 13300 6500
-Wire Wire Line
-	6600 3900 7100 3900
-Wire Wire Line
-	6600 4000 7100 4000
-Wire Wire Line
-	6600 4750 7100 4750
-Wire Wire Line
-	6600 4850 7100 4850
-Wire Wire Line
-	6000 5850 7100 5850
-Wire Wire Line
-	6000 5950 7100 5950
-Wire Wire Line
-	4450 2950 4450 4100
-Connection ~ 4450 4000
-Connection ~ 4450 3900
-Connection ~ 4450 3800
-Connection ~ 4450 3600
-Connection ~ 4450 3700
-Connection ~ 4450 3500
 $Sheet
 S 5200 8300 1450 1900
@@
 F7 "cfc6" O R 6650 9400 60
 $EndSheet
-Wire Wire Line
-	6650 8450 7100 8450
-Wire Wire Line
-	7100 8600 6650 8600
-Wire Wire Line
-	6650 8800 7100 8800
-Wire Wire Line
-	7100 9000 6650 9000
-Wire Wire Line
-	6650 9200 7100 9200
-Wire Wire Line
-	7100 9400 6650 9400
 $Sheet
 S 5200 10650 1450 900
@@
 F4 "c_couleurR" O R 6650 10900 60
 $EndSheet
-Wire Wire Line
-	6650 11050 7100 11050
-Wire Wire Line
-	7100 11200 6650 11200
-Wire Wire Line
-	6000 5750 6600 5750
-Wire Wire Line
-	6600 5750 6600 5400
-Wire Wire Line
-	7100 6750 6650 6750
-Wire Wire Line
-	6650 6900 7100 6900
-Wire Wire Line
-	7100 7050 6650 7050
-Wire Wire Line
-	6650 7200 7100 7200
-Wire Wire Line
-	7100 7350 6650 7350
-Wire Wire Line
-	13300 5150 13850 5150
-Wire Wire Line
-	13300 9600 13900 9600
-Wire Wire Line
-	13300 9900 13900 9900
-Wire Wire Line
-	6650 10900 7100 10900
-Wire Wire Line
-	6650 6600 7100 6600
 $Sheet
 S 7100 3650 6200 9800
@@
 F19 "TX-Pi" O L 7100 3900 60
 F20 "RX-Pi" I L 7100 4000 60
-F21 "TX-cervo" O L 7100 4750 60
-F22 "RX-cervo" I L 7100 4850 60
+F21 "TX-servo" O L 7100 4750 60
+F22 "RX-servo" I L 7100 4850 60
 F23 "Tx-balise" O L 7100 5850 60
 F24 "Rx-balise" I L 7100 5950 60
@@
 F35 "c_couleurG" I L 7100 11050 60
 F36 "c_couleurB" I L 7100 11200 60
-F37 "speed-cc" I L 7100 6250 60
-F38 "enable-cc" I L 7100 6350 60
-F39 "dir-cc" I L 7100 6150 60
-F40 "c-distance1" I L 7100 6600 60
-F41 "c-distance2" I L 7100 6750 60
-F42 "c-distance3" I L 7100 6900 60
-F43 "pince-M0" O R 13300 5150 60
-F44 "enable-cc" O R 13300 9300 60
-F45 "speed-cc" O R 13300 9600 60
-F46 "dir-cc" O R 13300 9900 60
-F47 "led_fusée" O L 7100 12350 60
+F37 "c-distance1" I L 7100 6600 60
+F38 "c-distance2" I L 7100 6750 60
+F39 "c-distance3" I L 7100 6900 60
+F40 "pince-M0" O R 13300 5150 60
+F41 "enable-cc" O R 13300 9300 60
+F42 "speed-cc" O R 13300 9600 60
+F43 "dir-cc" O R 13300 9900 60
+F44 "led_fusée" O L 7100 12350 60
+F45 "dir-servo" O L 7100 4650 60
 $EndSheet
 $Sheet
@@
 F7 "c-distance6" O R 6650 7350 60
 $EndSheet
-Wire Wire Line
-	13300 9300 13900 9300
-$Comp
-L CONN_01X02 P?
+$Comp
+L CONN_01X02 P1
 U 1 1 58B3634A
 P 6200 12400
-F 0 "P?" H 6200 12550 50  0000 C CNN
-F 1 "CONN_01X02" V 6300 12400 50  0000 C CNN
-F 2 "" H 6200 12400 50  0000 C CNN
+F 0 "P1" H 6200 12550 50  0000 C CNN
+F 1 "led-fusée" V 6300 12400 50  0000 C CNN
+F 2 "Pin_Headers:Pin_Header_Straight_1x02_Pitch2.54mm" H 6200 12400 50  0001 C CNN
 F 3 "" H 6200 12400 50  0000 C CNN
 	1    6200 12400
 	-1   0    0    1
 $EndComp
-Wire Wire Line
-	7100 12350 6400 12350
-Wire Wire Line
-	6400 12450 6550 12450
-Wire Wire Line
-	6550 12450 6550 12700
-$Comp
-L R R?
+$Comp
+L R R16
 U 1 1 58B38556
 P 6550 12850
-F 0 "R?" V 6630 12850 50  0000 C CNN
+F 0 "R16" V 6630 12850 50  0000 C CNN
 F 1 "1k" V 6550 12850 50  0000 C CNN
-F 2 "" V 6480 12850 50  0000 C CNN
+F 2 "Discret:R4-LARGE_PADS" V 6480 12850 50  0001 C CNN
 F 3 "" H 6550 12850 50  0000 C CNN
 	1    6550 12850
 	1    0    0    -1
 $EndComp
-Wire Wire Line
-	6550 13000 6550 13100
-$Comp
-L GND #PWR03
+$Comp
+L GND #PWR02
 U 1 1 58B388BC
 P 6550 13100
-F 0 "#PWR03" H 6550 12850 50  0001 C CNN
+F 0 "#PWR02" H 6550 12850 50  0001 C CNN
 F 1 "GND" H 6550 12950 50  0000 C CNN
 F 2 "" H 6550 13100 50  0000 C CNN
@@
 	1    0    0    -1
 $EndComp
+$Sheet
+S 5250 4500 1350 600
+U 58B88669
+F0 "servo_part" 60
+F1 "servo_part.sch" 60
+F2 "RX-servo" O R 6600 4850 60
+F3 "TX-servo" I R 6600 4750 60
+F4 "dir-servo" O R 6600 4650 60
+$EndSheet
+Wire Wire Line
+	13300 4250 13850 4250
+Wire Wire Line
+	13300 4400 13850 4400
+Wire Wire Line
+	13300 4550 13850 4550
+Wire Wire Line
+	13850 4700 13300 4700
+Wire Wire Line
+	13300 4850 13850 4850
+Wire Wire Line
+	13850 5000 13300 5000
+Wire Wire Line
+	13850 5300 13300 5300
+Wire Wire Line
+	13300 5450 13850 5450
+Wire Wire Line
+	13300 7300 13850 7300
+Wire Wire Line
+	13850 7100 13300 7100
+Wire Wire Line
+	13300 6900 13850 6900
+Wire Wire Line
+	13850 6650 13300 6650
+Wire Wire Line
+	13300 5850 13850 5850
+Wire Wire Line
+	13300 6000 13850 6000
+Wire Wire Line
+	13850 6150 13300 6150
+Wire Wire Line
+	13300 6300 13850 6300
+Wire Wire Line
+	13850 6500 13300 6500
+Wire Wire Line
+	6600 3900 7100 3900
+Wire Wire Line
+	6000 5850 7100 5850
+Wire Wire Line
+	6000 5950 7100 5950
+Wire Wire Line
+	6650 8450 7100 8450
+Wire Wire Line
+	7100 8600 6650 8600
+Wire Wire Line
+	6650 8800 7100 8800
+Wire Wire Line
+	7100 9000 6650 9000
+Wire Wire Line
+	6650 9200 7100 9200
+Wire Wire Line
+	7100 9400 6650 9400
+Wire Wire Line
+	6650 11050 7100 11050
+Wire Wire Line
+	7100 11200 6650 11200
+Wire Wire Line
+	6000 5750 6600 5750
+Wire Wire Line
+	6600 5750 6600 5400
+Wire Wire Line
+	7100 6750 6650 6750
+Wire Wire Line
+	6650 6900 7100 6900
+Wire Wire Line
+	7100 7050 6650 7050
+Wire Wire Line
+	6650 7200 7100 7200
+Wire Wire Line
+	7100 7350 6650 7350
+Wire Wire Line
+	13300 5150 13850 5150
+Wire Wire Line
+	13300 9600 13900 9600
+Wire Wire Line
+	13300 9900 13900 9900
+Wire Wire Line
+	6650 10900 7100 10900
+Wire Wire Line
+	6650 6600 7100 6600
+Wire Wire Line
+	13300 9300 13900 9300
+Wire Wire Line
+	7100 12350 6400 12350
+Wire Wire Line
+	6400 12450 6550 12450
+Wire Wire Line
+	6550 12450 6550 12700
+Wire Wire Line
+	6550 13000 6550 13100
+Wire Wire Line
+	7100 4750 6600 4750
+Wire Wire Line
+	7100 4850 6600 4850
+Wire Wire Line
+	7100 4650 6600 4650
+Wire Wire Line
+	6600 4000 7100 4000
+$Comp
+L CONN_01X02 P3
+U 1 1 589450AF
+P 6400 3950
+F 0 "P3" H 6400 4100 50  0000 C CNN
+F 1 "uart-pi" V 6500 3950 50  0000 C CNN
+F 2 "Pin_Headers:Pin_Header_Straight_1x02_Pitch2.54mm" H 6400 3950 50  0001 C CNN
+F 3 "" H 6400 3950 50  0000 C CNN
+	1    6400 3950
+	-1   0    0    1
+$EndComp
+$Comp
+L CONN_01X04 P2
+U 1 1 58BB0B25
+P 5800 5900
+F 0 "P2" H 5800 6150 50  0000 C CNN
+F 1 "Balise" V 5900 5900 50  0000 C CNN
+F 2 "Pin_Headers:Pin_Header_Straight_1x04_Pitch2.54mm" H 5800 5900 50  0001 C CNN
+F 3 "" H 5800 5900 50  0000 C CNN
+	1    5800 5900
+	-1   0    0    1
+$EndComp
+Wire Wire Line
+	6000 6050 6600 6050
+Wire Wire Line
+	6600 6050 6600 6150
+$Comp
+L GND #PWR03
+U 1 1 58BB0E74
+P 6600 6150
+F 0 "#PWR03" H 6600 5900 50  0001 C CNN
+F 1 "GND" H 6600 6000 50  0000 C CNN
+F 2 "" H 6600 6150 50  0000 C CNN
+F 3 "" H 6600 6150 50  0000 C CNN
+	1    6600 6150
+	1    0    0    -1
+$EndComp

Commit message: fin PCB
Parts:
- removed P2: Balise, Pin_Headers:Pin_Header_Straight_1x04_Pitch2.54mm, symbol CONN_01X04
- renumbered P1 to P2, R16 to R1
Changed lines of the file:
@@
 EESchema Schematic File Version 2
+LIBS:carte-asser-1A-2016-2017-rescue
 LIBS:power
 LIBS:device
@@
 $Descr A2 23386 16535
 encoding utf-8
-Sheet 1 9
+Sheet 1 10
 Title ""
 Date ""
@@
 F18 "roue-M1" I L 13850 7100 60
 F19 "roue-M2" I L 13850 7300 60
+F20 "Carte_Fault_1" I L 13850 7500 60
+F21 "Carte_Fault_2" I L 13850 7700 60
 $EndSheet
 $Sheet
@@
 F1 "pwr_part.sch" 60
 $EndSheet
-$Comp
-L +15V #PWR01
-U 1 1 589D46CA
-P 6600 5400
-F 0 "#PWR01" H 6600 5250 50  0001 C CNN
-F 1 "+15V" H 6600 5540 50  0000 C CNN
-F 2 "" H 6600 5400 50  0000 C CNN
-F 3 "" H 6600 5400 50  0000 C CNN
-	1    6600 5400
-	1    0    0    -1
-$EndComp
 $Sheet
 S 5200 8300 1450 1900
@@
 F44 "led_fusée" O L 7100 12350 60
 F45 "dir-servo" O L 7100 4650 60
+F46 "Carte_Fault_1" O R 13300 7500 60
+F47 "Carte_Fault_2" O R 13300 7700 60
 $EndSheet
 $Sheet
@@
 $EndSheet
 $Comp
-L CONN_01X02 P1
+L CONN_01X02 P2
 U 1 1 58B3634A
 P 6200 12400
-F 0 "P1" H 6200 12550 50  0000 C CNN
+F 0 "P2" H 6200 12550 50  0000 C CNN
 F 1 "led-fusée" V 6300 12400 50  0000 C CNN
 F 2 "Pin_Headers:Pin_Header_Straight_1x02_Pitch2.54mm" H 6200 12400 50  0001 C CNN
@@
 $EndComp
 $Comp
-L R R16
+L R R1
 U 1 1 58B38556
 P 6550 12850
-F 0 "R16" V 6630 12850 50  0000 C CNN
+F 0 "R1" V 6630 12850 50  0000 C CNN
 F 1 "1k" V 6550 12850 50  0000 C CNN
 F 2 "Discret:R4-LARGE_PADS" V 6480 12850 50  0001 C CNN
@@
 $EndComp
 $Comp
-L GND #PWR02
+L GND #PWR01
 U 1 1 58B388BC
 P 6550 13100
-F 0 "#PWR02" H 6550 12850 50  0001 C CNN
+F 0 "#PWR01" H 6550 12850 50  0001 C CNN
 F 1 "GND" H 6550 12950 50  0000 C CNN
 F 2 "" H 6550 13100 50  0000 C CNN
@@
 	6600 3900 7100 3900
 Wire Wire Line
-	6000 5850 7100 5850
-Wire Wire Line
-	6000 5950 7100 5950
-Wire Wire Line
 	6650 8450 7100 8450
 Wire Wire Line
@@
 Wire Wire Line
 	7100 11200 6650 11200
-Wire Wire Line
-	6000 5750 6600 5750
-Wire Wire Line
-	6600 5750 6600 5400
 Wire Wire Line
 	7100 6750 6650 6750
@@
 	-1   0    0    1
 $EndComp
-$Comp
-L CONN_01X04 P2
-U 1 1 58BB0B25
-P 5800 5900
-F 0 "P2" H 5800 6150 50  0000 C CNN
-F 1 "Balise" V 5900 5900 50  0000 C CNN
-F 2 "Pin_Headers:Pin_Header_Straight_1x04_Pitch2.54mm" H 5800 5900 50  0001 C CNN
-F 3 "" H 5800 5900 50  0000 C CNN
-	1    5800 5900
-	-1   0    0    1
-$EndComp
-Wire Wire Line
-	6000 6050 6600 6050
-Wire Wire Line
-	6600 6050 6600 6150
-$Comp
-L GND #PWR03
-U 1 1 58BB0E74
-P 6600 6150
-F 0 "#PWR03" H 6600 5900 50  0001 C CNN
-F 1 "GND" H 6600 6000 50  0000 C CNN
-F 2 "" H 6600 6150 50  0000 C CNN
-F 3 "" H 6600 6150 50  0000 C CNN
-	1    6600 6150
-	1    0    0    -1
-$EndComp
+Wire Wire Line
+	13300 7500 13850 7500
+Wire Wire Line
+	13300 7700 13850 7700
+$Sheet
+S 5250 5650 1350 550
+U 58D47F79
+F0 "balise_part" 60
+F1 "balise_part.sch" 60
+F2 "Tx-balise" I R 6600 5850 60
+F3 "Rx-balise" O R 6600 5950 60
+$EndSheet
+Wire Wire Line
+	6600 5950 7100 5950
+Wire Wire Line
+	7100 5850 6600 5850
 $EndSCHEMATC
