File: carte-asser-1A-2016-2017/cfc_part.sch (KiCad schematic (older format))
At the start: 12 parts, among them P16 CONN_01X02, P17 CONN_01X02, P18 CONN_01X02, P19 CONN_01X02, P20 CONN_01X02, P21 CONN_01X02

Commit message: PCB
Parts:
- P16: value CONN_01X02 -> cfc4; footprint (none) -> Pin_Headers:Pin_Header_Straight_1x02_Pitch2.54mm
- P17: value CONN_01X02 -> cfc1; footprint (none) -> Pin_Headers:Pin_Header_Straight_1x02_Pitch2.54mm
- P18: value CONN_01X02 -> cfc5; footprint (none) -> Pin_Headers:Pin_Header_Straight_1x02_Pitch2.54mm
- P19: value CONN_01X02 -> cfc2; footprint (none) -> Pin_Headers:Pin_Header_Straight_1x02_Pitch2.54mm
- P20: value CONN_01X02 -> cfc3; footprint (none) -> Pin_Headers:Pin_Header_Straight_1x02_Pitch2.54mm
- P21: value CONN_01X02 -> cfc6; footprint (none) -> Pin_Headers:Pin_Header_Straight_1x02_Pitch2.54mm
- R4, R5, R6, R7, R8, R9: footprint (none) -> Discret:R4-LARGE_PADS
Changed lines of the file:
@@
 $Descr A4 11693 8268
 encoding utf-8
-Sheet 5 8
+Sheet 5 9
 Title ""
 Date ""
@@
 P 3100 1700
 F 0 "P17" H 3100 1850 50  0000 C CNN
-F 1 "CONN_01X02" V 3200 1700 50  0000 C CNN
-F 2 "" H 3100 1700 50  0000 C CNN
+F 1 "cfc1" V 3200 1700 50  0000 C CNN
+F 2 "Pin_Headers:Pin_Header_Straight_1x02_Pitch2.54mm" H 3100 1700 50  0001 C CNN
 F 3 "" H 3100 1700 50  0000 C CNN
 	1    3100 1700
@@
 F 0 "R5" V 2280 2050 50  0000 C CNN
 F 1 "10k" V 2200 2050 50  0000 C CNN
-F 2 "" V 2130 2050 50  0000 C CNN
+F 2 "Discret:R4-LARGE_PADS" V 2130 2050 50  0001 C CNN
 F 3 "" H 2200 2050 50  0000 C CNN
 	1    2200 2050
@@
 P 5750 1600
 F 0 "P19" H 5750 1750 50  0000 C CNN
-F 1 "CONN_01X02" V 5850 1600 50  0000 C CNN
-F 2 "" H 5750 1600 50  0000 C CNN
+F 1 "cfc2" V 5850 1600 50  0000 C CNN
+F 2 "Pin_Headers:Pin_Header_Straight_1x02_Pitch2.54mm" H 5750 1600 50  0001 C CNN
 F 3 "" H 5750 1600 50  0000 C CNN
 	1    5750 1600
@@
 F 0 "R7" V 4930 1950 50  0000 C CNN
 F 1 "10k" V 4850 1950 50  0000 C CNN
-F 2 "" V 4780 1950 50  0000 C CNN
+F 2 "Discret:R4-LARGE_PADS" V 4780 1950 50  0001 C CNN
 F 3 "" H 4850 1950 50  0000 C CNN
 	1    4850 1950
@@
 P 8350 1500
 F 0 "P20" H 8350 1650 50  0000 C CNN
-F 1 "CONN_01X02" V 8450 1500 50  0000 C CNN
-F 2 "" H 8350 1500 50  0000 C CNN
+F 1 "cfc3" V 8450 1500 50  0000 C CNN
+F 2 "Pin_Headers:Pin_Header_Straight_1x02_Pitch2.54mm" H 8350 1500 50  0001 C CNN
 F 3 "" H 8350 1500 50  0000 C CNN
 	1    8350 1500
@@
 F 0 "R8" V 7530 1850 50  0000 C CNN
 F 1 "10k" V 7450 1850 50  0000 C CNN
-F 2 "" V 7380 1850 50  0000 C CNN
+F 2 "Discret:R4-LARGE_PADS" V 7380 1850 50  0001 C CNN
 F 3 "" H 7450 1850 50  0000 C CNN
 	1    7450 1850
@@
 P 2950 3800
 F 0 "P16" H 2950 3950 50  0000 C CNN
-F 1 "CONN_01X02" V 3050 3800 50  0000 C CNN
-F 2 "" H 2950 3800 50  0000 C CNN
+F 1 "cfc4" V 3050 3800 50  0000 C CNN
+F 2 "Pin_Headers:Pin_Header_Straight_1x02_Pitch2.54mm" H 2950 3800 50  0001 C CNN
 F 3 "" H 2950 3800 50  0000 C CNN
 	1    2950 3800
@@
 F 0 "R4" V 2130 4150 50  0000 C CNN
 F 1 "10k" V 2050 4150 50  0000 C CNN
-F 2 "" V 1980 4150 50  0000 C CNN
+F 2 "Discret:R4-LARGE_PADS" V 1980 4150 50  0001 C CNN
 F 3 "" H 2050 4150 50  0000 C CNN
 	1    2050 4150
@@
 P 5600 3650
 F 0 "P18" H 5600 3800 50  0000 C CNN
-F 1 "CONN_01X02" V 5700 3650 50  0000 C CNN
-F 2 "" H 5600 3650 50  0000 C CNN
+F 1 "cfc5" V 5700 3650 50  0000 C CNN
+F 2 "Pin_Headers:Pin_Header_Straight_1x02_Pitch2.54mm" H 5600 3650 50  0001 C CNN
 F 3 "" H 5600 3650 50  0000 C CNN
 	1    5600 3650
@@
 F 0 "R6" V 4780 4000 50  0000 C CNN
 F 1 "10k" V 4700 4000 50  0000 C CNN
-F 2 "" V 4630 4000 50  0000 C CNN
+F 2 "Discret:R4-LARGE_PADS" V 4630 4000 50  0001 C CNN
 F 3 "" H 4700 4000 50  0000 C CNN
 	1    4700 4000
@@
 P 8700 3700
 F 0 "P21" H 8700 3850 50  0000 C CNN
-F 1 "CONN_01X02" V 8800 3700 50  0000 C CNN
-F 2 "" H 8700 3700 50  0000 C CNN
+F 1 "cfc6" V 8800 3700 50  0000 C CNN
+F 2 "Pin_Headers:Pin_Header_Straight_1x02_Pitch2.54mm" H 8700 3700 50  0001 C CNN
 F 3 "" H 8700 3700 50  0000 C CNN
 	1    8700 3700
@@
 F 0 "R9" V 7880 4050 50  0000 C CNN
 F 1 "10k" V 7800 4050 50  0000 C CNN
-F 2 "" V 7730 4050 50  0000 C CNN
+F 2 "Discret:R4-LARGE_PADS" V 7730 4050 50  0001 C CNN
 F 3 "" H 7800 4050 50  0000 C CNN
 	1    7800 4050

Commit message: fin PCB
Parts:
- renumbered P17 to P10, P18 to P11, P19 to P12, P20 to P13, P21 to P14, P16 to P9, R9 to R10, R4 to R5, R5 to R6, R6 to R7, R7 to R8, R8 to R9
Changed lines of the file:
@@
 EESchema Schematic File Version 2
+LIBS:carte-asser-1A-2016-2017-rescue
 LIBS:power
 LIBS:device
@@
 $Descr A4 11693 8268
 encoding utf-8
-Sheet 5 9
+Sheet 5 10
 Title ""
 Date ""
@@
 $EndDescr
 $Comp
-L CONN_01X02 P17
+L CONN_01X02 P10
 U 1 1 58A0C256
 P 3100 1700
-F 0 "P17" H 3100 1850 50  0000 C CNN
+F 0 "P10" H 3100 1850 50  0000 C CNN
 F 1 "cfc1" V 3200 1700 50  0000 C CNN
 F 2 "Pin_Headers:Pin_Header_Straight_1x02_Pitch2.54mm" H 3100 1700 50  0001 C CNN
@@
 	2450 1650 2450 1300
 $Comp
-L +5V #PWR043
+L +5V #PWR041
 U 1 1 58A0C351
 P 2450 1300
-F 0 "#PWR043" H 2450 1150 50  0001 C CNN
+F 0 "#PWR041" H 2450 1150 50  0001 C CNN
 F 1 "+5V" H 2450 1440 50  0000 C CNN
 F 2 "" H 2450 1300 50  0000 C CNN
@@
 Connection ~ 2200 1750
 $Comp
-L R R5
+L R R6
 U 1 1 58A0C38D
 P 2200 2050
-F 0 "R5" V 2280 2050 50  0000 C CNN
+F 0 "R6" V 2280 2050 50  0000 C CNN
 F 1 "10k" V 2200 2050 50  0000 C CNN
 F 2 "Discret:R4-LARGE_PADS" V 2130 2050 50  0001 C CNN
@@
 	2200 2200 2200 2400
 $Comp
-L GND #PWR044
+L GND #PWR042
 U 1 1 58A0C3D4
 P 2200 2400
-F 0 "#PWR044" H 2200 2150 50  0001 C CNN
+F 0 "#PWR042" H 2200 2150 50  0001 C CNN
 F 1 "GND" H 2200 2250 50  0000 C CNN
 F 2 "" H 2200 2400 50  0000 C CNN
@@
 $EndComp
 $Comp
-L CONN_01X02 P19
+L CONN_01X02 P12
 U 1 1 58A0C574
 P 5750 1600
-F 0 "P19" H 5750 1750 50  0000 C CNN
+F 0 "P12" H 5750 1750 50  0000 C CNN
 F 1 "cfc2" V 5850 1600 50  0000 C CNN
 F 2 "Pin_Headers:Pin_Header_Straight_1x02_Pitch2.54mm" H 5750 1600 50  0001 C CNN
@@
 	5100 1550 5100 1200
 $Comp
-L +5V #PWR045
+L +5V #PWR043
 U 1 1 58A0C57C
 P 5100 1200
-F 0 "#PWR045" H 5100 1050 50  0001 C CNN
+F 0 "#PWR043" H 5100 1050 50  0001 C CNN
 F 1 "+5V" H 5100 1340 50  0000 C CNN
 F 2 "" H 5100 1200 50  0000 C CNN
@@
 Connection ~ 4850 1650
 $Comp
-L R R7
+L R R8
 U 1 1 58A0C586
 P 4850 1950
-F 0 "R7" V 4930 1950 50  0000 C CNN
+F 0 "R8" V 4930 1950 50  0000 C CNN
 F 1 "10k" V 4850 1950 50  0000 C CNN
 F 2 "Discret:R4-LARGE_PADS" V 4780 1950 50  0001 C CNN
@@
 	4850 2100 4850 2300
 $Comp
-L GND #PWR046
+L GND #PWR044
 U 1 1 58A0C58D
 P 4850 2300
-F 0 "#PWR046" H 4850 2050 50  0001 C CNN
+F 0 "#PWR044" H 4850 2050 50  0001 C CNN
 F 1 "GND" H 4850 2150 50  0000 C CNN
 F 2 "" H 4850 2300 50  0000 C CNN
@@
 $EndComp
 $Comp
-L CONN_01X02 P20
+L CONN_01X02 P13
 U 1 1 58A0C737
 P 8350 1500
-F 0 "P20" H 8350 1650 50  0000 C CNN
+F 0 "P13" H 8350 1650 50  0000 C CNN
 F 1 "cfc3" V 8450 1500 50  0000 C CNN
 F 2 "Pin_Headers:Pin_Header_Straight_1x02_Pitch2.54mm" H 8350 1500 50  0001 C CNN
@@
 	7700 1450 7700 1100
 $Comp
-L +5V #PWR047
+L +5V #PWR045
 U 1 1 58A0C73F
 P 7700 1100
-F 0 "#PWR047" H 7700 950 50  0001 C CNN
+F 0 "#PWR045" H 7700 950 50  0001 C CNN
 F 1 "+5V" H 7700 1240 50  0000 C CNN
 F 2 "" H 7700 1100 50  0000 C CNN
@@
 Connection ~ 7450 1550
 $Comp
-L R R8
+L R R9
 U 1 1 58A0C749
 P 7450 1850
-F 0 "R8" V 7530 1850 50  0000 C CNN
+F 0 "R9" V 7530 1850 50  0000 C CNN
 F 1 "10k" V 7450 1850 50  0000 C CNN
 F 2 "Discret:R4-LARGE_PADS" V 7380 1850 50  0001 C CNN
@@
 	7450 2000 7450 2200
 $Comp
-L GND #PWR048
+L GND #PWR046
 U 1 1 58A0C750
 P 7450 2200
-F 0 "#PWR048" H 7450 1950 50  0001 C CNN
+F 0 "#PWR046" H 7450 1950 50  0001 C CNN
 F 1 "GND" H 7450 2050 50  0000 C CNN
 F 2 "" H 7450 2200 50  0000 C CNN
@@
 $EndComp
 $Comp
-L CONN_01X02 P16
+L CONN_01X02 P9
 U 1 1 58A0C85E
 P 2950 3800
-F 0 "P16" H 2950 3950 50  0000 C CNN
+F 0 "P9" H 2950 3950 50  0000 C CNN
 F 1 "cfc4" V 3050 3800 50  0000 C CNN
 F 2 "Pin_Headers:Pin_Header_Straight_1x02_Pitch2.54mm" H 2950 3800 50  0001 C CNN
@@
 	2300 3750 2300 3400
 $Comp
-L +5V #PWR049
+L +5V #PWR047
 U 1 1 58A0C866
 P 2300 3400
-F 0 "#PWR049" H 2300 3250 50  0001 C CNN
+F 0 "#PWR047" H 2300 3250 50  0001 C CNN
 F 1 "+5V" H 2300 3540 50  0000 C CNN
 F 2 "" H 2300 3400 50  0000 C CNN
@@
 Connection ~ 2050 3850
 $Comp
-L R R4
+L R R5
 U 1 1 58A0C870
 P 2050 4150
-F 0 "R4" V 2130 4150 50  0000 C CNN
+F 0 "R5" V 2130 4150 50  0000 C CNN
 F 1 "10k" V 2050 4150 50  0000 C CNN
 F 2 "Discret:R4-LARGE_PADS" V 1980 4150 50  0001 C CNN
@@
 	2050 4300 2050 4500
 $Comp
-L GND #PWR050
+L GND #PWR048
 U 1 1 58A0C877
 P 2050 4500
-F 0 "#PWR050" H 2050 4250 50  0001 C CNN
+F 0 "#PWR048" H 2050 4250 50  0001 C CNN
 F 1 "GND" H 2050 4350 50  0000 C CNN
 F 2 "" H 2050 4500 50  0000 C CNN
@@
 $EndComp
 $Comp
-L CONN_01X02 P18
+L CONN_01X02 P11
 U 1 1 58A0C9D1
 P 5600 3650
-F 0 "P18" H 5600 3800 50  0000 C CNN
+F 0 "P11" H 5600 3800 50  0000 C CNN
 F 1 "cfc5" V 5700 3650 50  0000 C CNN
 F 2 "Pin_Headers:Pin_Header_Straight_1x02_Pitch2.54mm" H 5600 3650 50  0001 C CNN
@@
 	4950 3600 4950 3250
 $Comp
-L +5V #PWR051
+L +5V #PWR049
 U 1 1 58A0C9D9
 P 4950 3250
-F 0 "#PWR051" H 4950 3100 50  0001 C CNN
+F 0 "#PWR049" H 4950 3100 50  0001 C CNN
 F 1 "+5V" H 4950 3390 50  0000 C CNN
 F 2 "" H 4950 3250 50  0000 C CNN
@@
 Connection ~ 4700 3700
 $Comp
-L R R6
+L R R7
 U 1 1 58A0C9E3
 P 4700 4000
-F 0 "R6" V 4780 4000 50  0000 C CNN
+F 0 "R7" V 4780 4000 50  0000 C CNN
 F 1 "10k" V 4700 4000 50  0000 C CNN
 F 2 "Discret:R4-LARGE_PADS" V 4630 4000 50  0001 C CNN
@@
 	4700 4150 4700 4350
 $Comp
-L GND #PWR052
+L GND #PWR050
 U 1 1 58A0C9EA
 P 4700 4350
-F 0 "#PWR052" H 4700 4100 50  0001 C CNN
+F 0 "#PWR050" H 4700 4100 50  0001 C CNN
 F 1 "GND" H 4700 4200 50  0000 C CNN
 F 2 "" H 4700 4350 50  0000 C CNN
@@
 $EndComp
 $Comp
-L CONN_01X02 P21
+L CONN_01X02 P14
 U 1 1 58A0CAE4
 P 8700 3700
-F 0 "P21" H 8700 3850 50  0000 C CNN
+F 0 "P14" H 8700 3850 50  0000 C CNN
 F 1 "cfc6" V 8800 3700 50  0000 C CNN
 F 2 "Pin_Headers:Pin_Header_Straight_1x02_Pitch2.54mm" H 8700 3700 50  0001 C CNN
@@
 	8050 3650 8050 3300
 $Comp
-L +5V #PWR053
+L +5V #PWR051
 U 1 1 58A0CAEC
 P 8050 3300
-F 0 "#PWR053" H 8050 3150 50  0001 C CNN
+F 0 "#PWR051" H 8050 3150 50  0001 C CNN
 F 1 "+5V" H 8050 3440 50  0000 C CNN
 F 2 "" H 8050 3300 50  0000 C CNN
@@
 Connection ~ 7800 3750
 $Comp
-L R R9
+L R R10
 U 1 1 58A0CAF6
 P 7800 4050
-F 0 "R9" V 7880 4050 50  0000 C CNN
+F 0 "R10" V 7880 4050 50  0000 C CNN
 F 1 "10k" V 7800 4050 50  0000 C CNN
 F 2 "Discret:R4-LARGE_PADS" V 7730 4050 50  0001 C CNN
@@
 	7800 4200 7800 4400
 $Comp
-L GND #PWR054
+L GND #PWR052
 U 1 1 58A0CAFD
 P 7800 4400
-F 0 "#PWR054" H 7800 4150 50  0001 C CNN
+F 0 "#PWR052" H 7800 4150 50  0001 C CNN
 F 1 "GND" H 7800 4250 50  0000 C CNN
 F 2 "" H 7800 4400 50  0000 C CNN
