File: carte-asser-1A-2016-2017/command_part.sch (KiCad schematic (older format))
At the start: 1 part

Commit message: Fin PCB
Parts:
- gave numbers to parts that had none: 1
Connections:
- net c_couleurB: now reaches U9.22 (PC1)
- net c_couleurG: now reaches U9.25 (PA1)
- net c_couleurR: now reaches U9.26 (PA0)
- net led_fusée: now reaches U9.74 (PA5)
Changed lines of the file:
@@
 LIBS:valves
 LIBS:robot_1A
-LIBS:carte-asser-1A-cache
 LIBS:carte-asser-1A-2016-2017-cache
 EELAYER 25 0
@@
 $Descr A2 23386 16535
 encoding utf-8
-Sheet 5 7
+Sheet 7 8
 Title ""
 Date ""
@@
 $EndDescr
 $Comp
-L Nucleo-64 U?
+L Nucleo-64 U9
 U 1 1 5893E3C6
 P 7600 14450
-F 0 "U?" H 7650 14500 60  0000 C CNN
+F 0 "U9" H 7650 14500 60  0000 C CNN
 F 1 "Nucleo-64" H 11950 23450 100 0000 C CNN
 F 2 "" H 11850 25900 60  0001 C CNN
@@
 Wire Wire Line
 	15750 9850 16350 9850
-Text HLabel 16350 9850 2    60   Input ~ 0
+Text HLabel 16350 9850 2    60   Output ~ 0
 speed-cc
 Wire Wire Line
 	15750 10050 16350 10050
-Text HLabel 16350 10050 2    60   Input ~ 0
+Text HLabel 16350 10050 2    60   Output ~ 0
 enable-cc
 Wire Wire Line
 	15750 9650 16350 9650
-Text HLabel 16350 9650 2    60   Input ~ 0
+Text HLabel 16350 9650 2    60   Output ~ 0
 dir-cc
-Text HLabel 16350 3850 2    60   Input ~ 0
+Text HLabel 16350 3850 2    60   Output ~ 0
 enable-p1
 Wire Wire Line
-	15750 3850 16350 3850
-Wire Wire Line
 	15750 4050 16350 4050
-Text HLabel 16350 4050 2    60   Input ~ 0
+Text HLabel 16350 4050 2    60   Output ~ 0
 enable-p2
-Wire Wire Line
-	15750 4250 16350 4250
-Text HLabel 16350 4250 2    60   Input ~ 0
+Text HLabel 16350 4250 2    60   Output ~ 0
 step-p1
-Text HLabel 16350 4850 2    60   Input ~ 0
+Text HLabel 16350 4850 2    60   Output ~ 0
 step-p2
-Text HLabel 16350 5050 2    60   Input ~ 0
+Text HLabel 16350 5050 2    60   Output ~ 0
 dir-p1
-Text HLabel 16350 5250 2    60   Input ~ 0
+Text HLabel 16350 5250 2    60   Output ~ 0
 dir-p2
-Text HLabel 16350 5450 2    60   Input ~ 0
+Text HLabel 16350 5450 2    60   Output ~ 0
 pince-M0
-Text HLabel 16350 5850 2    60   Input ~ 0
+Text HLabel 16350 5850 2    60   Output ~ 0
 pince-M1
-Text HLabel 16350 6050 2    60   Input ~ 0
+Text HLabel 16350 6050 2    60   Output ~ 0
 pince-M2
 Wire Wire Line
-	15750 4850 16350 4850
-Wire Wire Line
 	15750 5050 16350 5050
 Wire Wire Line
@@
 	17350 5650 17350 5900
 $Comp
-L GND #PWR044
+L GND #PWR072
 U 1 1 589476FA
 P 17350 5900
-F 0 "#PWR044" H 17350 5650 50  0001 C CNN
+F 0 "#PWR072" H 17350 5650 50  0001 C CNN
 F 1 "GND" H 17350 5750 50  0000 C CNN
 F 2 "" H 17350 5900 50  0000 C CNN
@@
 	17100 8850 17100 9050
 $Comp
-L GND #PWR045
+L GND #PWR073
 U 1 1 5894773B
 P 17100 9050
-F 0 "#PWR045" H 17100 8800 50  0001 C CNN
+F 0 "#PWR073" H 17100 8800 50  0001 C CNN
 F 1 "GND" H 17100 8900 50  0000 C CNN
 F 2 "" H 17100 9050 50  0000 C CNN
@@
 	6850 5650 6850 5950
 $Comp
-L GND #PWR046
+L GND #PWR074
 U 1 1 5894779E
 P 6850 5950
-F 0 "#PWR046" H 6850 5700 50  0001 C CNN
+F 0 "#PWR074" H 6850 5700 50  0001 C CNN
 F 1 "GND" H 6850 5800 50  0000 C CNN
 F 2 "" H 6850 5950 50  0000 C CNN
@@
 	8450 10250 8650 10250
 $Comp
-L GND #PWR047
+L GND #PWR075
 U 1 1 58947867
 P 8250 8850
-F 0 "#PWR047" H 8250 8600 50  0001 C CNN
+F 0 "#PWR075" H 8250 8600 50  0001 C CNN
 F 1 "GND" H 8250 8700 50  0000 C CNN
 F 2 "" H 8250 8850 50  0000 C CNN
@@
 $EndComp
 $Comp
-L GND #PWR048
+L GND #PWR076
 U 1 1 5894787D
 P 8450 10250
-F 0 "#PWR048" H 8450 10000 50  0001 C CNN
+F 0 "#PWR076" H 8450 10000 50  0001 C CNN
 F 1 "GND" H 8450 10100 50  0000 C CNN
 F 2 "" H 8450 10250 50  0000 C CNN
@@
 $EndComp
 Wire Wire Line
-	15750 6250 16400 6250
-Wire Wire Line
 	15750 6450 16400 6450
 Wire Wire Line
@@
 Wire Wire Line
 	15750 9450 16400 9450
-Text HLabel 16400 6250 2    60   Input ~ 0
+Text HLabel 16400 6250 2    60   Output ~ 0
 enable-r1
-Text HLabel 16400 6450 2    60   Input ~ 0
+Text HLabel 16400 6450 2    60   Output ~ 0
 enable-r2
-Text HLabel 16400 6650 2    60   Input ~ 0
+Text HLabel 16400 6650 2    60   Output ~ 0
 step-r1
-Text HLabel 16400 7050 2    60   Input ~ 0
+Text HLabel 16400 7050 2    60   Output ~ 0
 step-r2
-Text HLabel 16400 8050 2    60   Input ~ 0
+Text HLabel 16400 8050 2    60   Output ~ 0
 dir-r1
-Text HLabel 16400 8250 2    60   Input ~ 0
+Text HLabel 16400 8250 2    60   Output ~ 0
 dir-r2
-Text HLabel 16400 8450 2    60   Input ~ 0
+Text HLabel 16400 8450 2    60   Output ~ 0
 roue-M0
-Text HLabel 16400 9250 2    60   Input ~ 0
+Text HLabel 16400 9250 2    60   Output ~ 0
 roue-M1
-Text HLabel 16400 9450 2    60   Input ~ 0
+Text HLabel 16400 9450 2    60   Output ~ 0
 roue-M2
 Wire Wire Line
@@
 	7200 8450 7200 8200
 $Comp
-L +5V #PWR?
+L +5V #PWR077
 U 1 1 589E3F8C
 P 7200 8200
-F 0 "#PWR?" H 7200 8050 50  0001 C CNN
+F 0 "#PWR077" H 7200 8050 50  0001 C CNN
 F 1 "+5V" H 7200 8340 50  0000 C CNN
 F 2 "" H 7200 8200 50  0000 C CNN
@@
 Wire Wire Line
 	15750 11250 16400 11250
+Wire Wire Line
+	8650 10850 7750 10850
+Text HLabel 7750 10850 0    60   Input ~ 0
+c_couleurR
+Wire Wire Line
+	8650 11050 7750 11050
+Wire Wire Line
+	8650 11650 7750 11650
+Text HLabel 7750 11050 0    60   Input ~ 0
+c_couleurG
+Text HLabel 7750 11650 0    60   Input ~ 0
+c_couleurB
+Wire Wire Line
+	15750 6250 16400 6250
+Wire Wire Line
+	15750 4850 16350 4850
+Wire Wire Line
+	15750 4250 16350 4250
+Wire Wire Line
+	15750 3850 16350 3850
+Wire Wire Line
+	15750 9050 16350 9050
+Text HLabel 16350 9050 2    60   Output ~ 0
+led_fusée
 $EndSCHEMATC

Commit message: PCB
Parts:
- U9: footprint (none) -> robot_1A:Nucleo-64
Connections:
- net dir-servo: now reaches U9.2 (PC2)
- net RX-cervo renamed RX-servo
- net TX-cervo renamed TX-servo
Changed lines of the file:
@@
 $Descr A2 23386 16535
 encoding utf-8
-Sheet 7 8
+Sheet 7 9
 Title ""
 Date ""
@@
 F 0 "U9" H 7650 14500 60  0000 C CNN
 F 1 "Nucleo-64" H 11950 23450 100 0000 C CNN
-F 2 "" H 11850 25900 60  0001 C CNN
+F 2 "robot_1A:Nucleo-64" H 11850 25900 60  0001 C CNN
 F 3 "" H 11850 25900 60  0001 C CNN
 	1    7600 14450
@@
 	17350 5650 17350 5900
 $Comp
-L GND #PWR072
+L GND #PWR068
 U 1 1 589476FA
 P 17350 5900
-F 0 "#PWR072" H 17350 5650 50  0001 C CNN
+F 0 "#PWR068" H 17350 5650 50  0001 C CNN
 F 1 "GND" H 17350 5750 50  0000 C CNN
 F 2 "" H 17350 5900 50  0000 C CNN
@@
 	17100 8850 17100 9050
 $Comp
-L GND #PWR073
+L GND #PWR069
 U 1 1 5894773B
 P 17100 9050
-F 0 "#PWR073" H 17100 8800 50  0001 C CNN
+F 0 "#PWR069" H 17100 8800 50  0001 C CNN
 F 1 "GND" H 17100 8900 50  0000 C CNN
 F 2 "" H 17100 9050 50  0000 C CNN
@@
 	6850 5650 6850 5950
 $Comp
-L GND #PWR074
+L GND #PWR070
 U 1 1 5894779E
 P 6850 5950
-F 0 "#PWR074" H 6850 5700 50  0001 C CNN
+F 0 "#PWR070" H 6850 5700 50  0001 C CNN
 F 1 "GND" H 6850 5800 50  0000 C CNN
 F 2 "" H 6850 5950 50  0000 C CNN
@@
 	8450 10250 8650 10250
 $Comp
-L GND #PWR075
+L GND #PWR071
 U 1 1 58947867
 P 8250 8850
-F 0 "#PWR075" H 8250 8600 50  0001 C CNN
+F 0 "#PWR071" H 8250 8600 50  0001 C CNN
 F 1 "GND" H 8250 8700 50  0000 C CNN
 F 2 "" H 8250 8850 50  0000 C CNN
@@
 $EndComp
 $Comp
-L GND #PWR076
+L GND #PWR072
 U 1 1 5894787D
 P 8450 10250
-F 0 "#PWR076" H 8450 10000 50  0001 C CNN
+F 0 "#PWR072" H 8450 10000 50  0001 C CNN
 F 1 "GND" H 8450 10100 50  0000 C CNN
 F 2 "" H 8450 10250 50  0000 C CNN
@@
 Wire Wire Line
 	8650 3850 8250 3850
-Wire Wire Line
-	8650 5050 8200 5050
 Text HLabel 8250 4050 0    60   Output ~ 0
-TX-cervo
+TX-servo
 Text HLabel 8150 8250 0    60   Input ~ 0
-RX-cervo
+RX-servo
 Text HLabel 8250 3850 0    60   Output ~ 0
 Tx-balise
@@
 	7200 8450 7200 8200
 $Comp
-L +5V #PWR077
+L +5V #PWR073
 U 1 1 589E3F8C
 P 7200 8200
-F 0 "#PWR077" H 7200 8050 50  0001 C CNN
+F 0 "#PWR073" H 7200 8050 50  0001 C CNN
 F 1 "+5V" H 7200 8340 50  0000 C CNN
 F 2 "" H 7200 8200 50  0000 C CNN
@@
 Text HLabel 16350 9050 2    60   Output ~ 0
 led_fusée
+Wire Wire Line
+	8650 7250 7750 7250
+Text HLabel 7750 7250 0    60   Input ~ 0
+dir-servo
 $EndSCHEMATC

Commit message: fin PCB
Parts:
- renumbered U9 to U10
Connections:
- net +5V: now also U10.37 (E5V); no longer U10.38 (PD2)
- net GND: no longer U10.37 (E5V)
- net RX-servo: now also U10.38 (PD2); no longer U10.39 (PC11)
- net Rx-balise: now also U10.39 (PC11); no longer U10.40 (NC)
- net dir-p1: now also U10.74 (PA5); no longer U10.53 (PA11)
- net dir-p2: now also U10.78 (PB8); no longer U10.52 (PB12)
- net dir-r1: now also U10.47 (PB15); no longer U10.79 (PC9)
- net dir-r2: now also U10.43 (PC4); no longer U10.78 (PB8)
- net enable-p2: now also U10.54 (PA12); no longer U10.58 (PC6)
- net enable-r1: now also U10.53 (PA11); no longer U10.47 (PB15)
- net led_fusée: now also U10.79 (PC9); no longer U10.74 (PA5)
- net pince-M0: now also U10.72 (PA7); no longer U10.51 (PB11)
- net pince-M1: now also U10.58 (PC6); no longer U10.49 (PB2)
- net pince-M2: now also U10.73 (PA6); no longer U10.48 (PB1)
- net roue-M0: now also U10.52 (PB12); no longer U10.77 (PB9)
- net roue-M1: now also U10.51 (PB11); no longer U10.73 (PA6)
- net roue-M2: now also U10.49 (PB2); no longer U10.72 (PA7)
- net step-p2: now also U10.77 (PB9); no longer U10.54 (PA12)
- net step-r1: now also U10.48 (PB1); no longer U10.45 (PB13)
- net step-r2: now also U10.45 (PB13); no longer U10.43 (PC4)
- net Carte_Fault_2: now reaches U10.61 (PA3)
- net Carte_Fault_1: now reaches U10.62 (PA2)
- no-connect marks 0 -> 26
Changed lines of the file:
@@
 EESchema Schematic File Version 2
+LIBS:carte-asser-1A-2016-2017-rescue
 LIBS:power
 LIBS:device
@@
 $Descr A2 23386 16535
 encoding utf-8
-Sheet 7 9
+Sheet 7 10
 Title ""
 Date ""
@@
 $EndDescr
 $Comp
-L Nucleo-64 U9
+L Nucleo-64 U10
 U 1 1 5893E3C6
 P 7600 14450
-F 0 "U9" H 7650 14500 60  0000 C CNN
+F 0 "U10" H 7650 14500 60  0000 C CNN
 F 1 "Nucleo-64" H 11950 23450 100 0000 C CNN
 F 2 "robot_1A:Nucleo-64" H 11850 25900 60  0001 C CNN
@@
 Wire Wire Line
 	15750 4050 16350 4050
-Text HLabel 16350 4050 2    60   Output ~ 0
+Text HLabel 16350 4850 2    60   Output ~ 0
 enable-p2
 Text HLabel 16350 4250 2    60   Output ~ 0
 step-p1
-Text HLabel 16350 4850 2    60   Output ~ 0
+Text HLabel 16400 8450 2    60   Output ~ 0
 step-p2
-Text HLabel 16350 5050 2    60   Output ~ 0
+Text HLabel 16350 9050 2    60   Output ~ 0
 dir-p1
-Text HLabel 16350 5250 2    60   Output ~ 0
+Text HLabel 16400 8250 2    60   Output ~ 0
 dir-p2
-Text HLabel 16350 5450 2    60   Output ~ 0
+Text HLabel 16400 9450 2    60   Output ~ 0
 pince-M0
-Text HLabel 16350 5850 2    60   Output ~ 0
+Text HLabel 16350 4050 2    60   Output ~ 0
 pince-M1
-Text HLabel 16350 6050 2    60   Output ~ 0
+Text HLabel 16400 9250 2    60   Output ~ 0
 pince-M2
 Wire Wire Line
@@
 	17350 5650 17350 5900
 $Comp
-L GND #PWR068
+L GND #PWR066
 U 1 1 589476FA
 P 17350 5900
-F 0 "#PWR068" H 17350 5650 50  0001 C CNN
+F 0 "#PWR066" H 17350 5650 50  0001 C CNN
 F 1 "GND" H 17350 5750 50  0000 C CNN
 F 2 "" H 17350 5900 50  0000 C CNN
@@
 	17100 8850 17100 9050
 $Comp
-L GND #PWR069
+L GND #PWR067
 U 1 1 5894773B
 P 17100 9050
-F 0 "#PWR069" H 17100 8800 50  0001 C CNN
+F 0 "#PWR067" H 17100 8800 50  0001 C CNN
 F 1 "GND" H 17100 8900 50  0000 C CNN
 F 2 "" H 17100 9050 50  0000 C CNN
@@
 	6850 5650 6850 5950
 $Comp
-L GND #PWR070
+L GND #PWR068
 U 1 1 5894779E
 P 6850 5950
-F 0 "#PWR070" H 6850 5700 50  0001 C CNN
+F 0 "#PWR068" H 6850 5700 50  0001 C CNN
 F 1 "GND" H 6850 5800 50  0000 C CNN
 F 2 "" H 6850 5950 50  0000 C CNN
@@
 	8650 8850 8250 8850
 Wire Wire Line
-	8250 8850 8250 8650
-Wire Wire Line
 	8450 10250 8650 10250
 $Comp
-L GND #PWR071
+L GND #PWR069
 U 1 1 58947867
 P 8250 8850
-F 0 "#PWR071" H 8250 8600 50  0001 C CNN
+F 0 "#PWR069" H 8250 8600 50  0001 C CNN
 F 1 "GND" H 8250 8700 50  0000 C CNN
 F 2 "" H 8250 8850 50  0000 C CNN
@@
 $EndComp
 $Comp
-L GND #PWR072
+L GND #PWR070
 U 1 1 5894787D
 P 8450 10250
-F 0 "#PWR072" H 8450 10000 50  0001 C CNN
+F 0 "#PWR070" H 8450 10000 50  0001 C CNN
 F 1 "GND" H 8450 10100 50  0000 C CNN
 F 2 "" H 8450 10250 50  0000 C CNN
@@
 Wire Wire Line
 	15750 9450 16400 9450
-Text HLabel 16400 6250 2    60   Output ~ 0
+Text HLabel 16350 5050 2    60   Output ~ 0
 enable-r1
 Text HLabel 16400 6450 2    60   Output ~ 0
 enable-r2
+Text HLabel 16350 6050 2    60   Output ~ 0
+step-r1
 Text HLabel 16400 6650 2    60   Output ~ 0
-step-r1
+step-r2
+Text HLabel 16400 6250 2    60   Output ~ 0
+dir-r1
 Text HLabel 16400 7050 2    60   Output ~ 0
-step-r2
-Text HLabel 16400 8050 2    60   Output ~ 0
-dir-r1
-Text HLabel 16400 8250 2    60   Output ~ 0
 dir-r2
-Text HLabel 16400 8450 2    60   Output ~ 0
+Text HLabel 16350 5250 2    60   Output ~ 0
 roue-M0
-Text HLabel 16400 9250 2    60   Output ~ 0
+Text HLabel 16350 5450 2    60   Output ~ 0
 roue-M1
-Text HLabel 16400 9450 2    60   Output ~ 0
+Text HLabel 16350 5850 2    60   Output ~ 0
 roue-M2
 Wire Wire Line
@@
 Text HLabel 8250 4050 0    60   Output ~ 0
 TX-servo
-Text HLabel 8150 8250 0    60   Input ~ 0
+Text HLabel 8150 8450 0    60   Input ~ 0
 RX-servo
 Text HLabel 8250 3850 0    60   Output ~ 0
 Tx-balise
-Wire Wire Line
-	8650 8050 8150 8050
-Text HLabel 8150 8050 0    60   Input ~ 0
+Text HLabel 8150 8250 0    60   Input ~ 0
 Rx-balise
 Wire Wire Line
@@
 	8450 10050 8650 10050
 Wire Wire Line
-	7200 8450 8650 8450
-Wire Wire Line
-	7200 8450 7200 8200
-$Comp
-L +5V #PWR073
+	7200 8200 7200 9250
+$Comp
+L +5V #PWR071
 U 1 1 589E3F8C
 P 7200 8200
-F 0 "#PWR073" H 7200 8050 50  0001 C CNN
+F 0 "#PWR071" H 7200 8050 50  0001 C CNN
 F 1 "+5V" H 7200 8340 50  0000 C CNN
 F 2 "" H 7200 8200 50  0000 C CNN
@@
 $EndComp
 Wire Wire Line
-	8250 8650 8650 8650
-Wire Wire Line
-	7900 8450 7900 9250
-Connection ~ 7900 8450
-Wire Wire Line
-	7900 9250 8650 9250
+	7200 9250 8650 9250
 Wire Wire Line
 	8650 4050 8250 4050
@@
 Wire Wire Line
 	15750 9050 16350 9050
-Text HLabel 16350 9050 2    60   Output ~ 0
+Text HLabel 16400 8050 2    60   Output ~ 0
 led_fusée
 Wire Wire Line
@@
 Text HLabel 7750 7250 0    60   Input ~ 0
 dir-servo
+Wire Wire Line
+	15750 11650 16400 11650
+Wire Wire Line
+	15750 11450 16400 11450
+Text HLabel 16400 11450 2    60   Input ~ 0
+Carte_Fault_1
+Text HLabel 16400 11650 2    60   Input ~ 0
+Carte_Fault_2
+Wire Wire Line
+	7200 8650 8650 8650
+Connection ~ 7200 8650
+Wire Wire Line
+	8650 8450 8150 8450
+NoConn ~ 8650 3650
+NoConn ~ 8650 4250
+NoConn ~ 8650 4450
+NoConn ~ 8650 4650
+NoConn ~ 8650 4850
+NoConn ~ 8650 5050
+NoConn ~ 8650 7050
+NoConn ~ 8650 7450
+NoConn ~ 8650 8050
+NoConn ~ 8650 9050
+NoConn ~ 8650 9450
+NoConn ~ 8650 9650
+NoConn ~ 8650 9850
+NoConn ~ 8650 10450
+NoConn ~ 8650 10650
+NoConn ~ 8650 11250
+NoConn ~ 8650 11450
+NoConn ~ 8650 11850
+NoConn ~ 15750 8650
+NoConn ~ 15750 7850
+NoConn ~ 15750 7450
+NoConn ~ 15750 7250
+NoConn ~ 15750 6850
+NoConn ~ 15750 4650
+NoConn ~ 15750 4450
+NoConn ~ 15750 3650
 $EndSCHEMATC
