File: carte-asser-1A-2016-2017/distance_captor_part.sch (KiCad schematic (older format))
At the start: 18 parts

Commit message: Fin PCB
Parts:
- removed D? (x12): D_Small, symbol D_Small
- gave numbers to parts that had none: 6
Connections:
- net +5V: now also P10.1 (P1), P11.1 (P1), P12.1 (P1), P13.1 (P1), P14.1 (P1), P15.1 (P1)
- net c-distance1: now also P10.2 (P2)
- net c-distance2: now also P13.2 (P2)
- net c-distance3: now also P14.2 (P2)
- net c-distance4: now also P11.2 (P2)
- net c-distance5: now also P12.2 (P2)
- net c-distance6: now also P15.2 (P2)

Commit message: PCB
Parts:
- P10: value CONN_01X03 -> dist-capt1; footprint (none) -> Pin_Headers:Pin_Header_Straight_1x03_Pitch2.54mm
- P11: value CONN_01X03 -> dist-capt4; footprint (none) -> Pin_Headers:Pin_Header_Straight_1x03_Pitch2.54mm
- P12: value CONN_01X03 -> dist-capt5; footprint (none) -> Pin_Headers:Pin_Header_Straight_1x03_Pitch2.54mm
- P13: value CONN_01X03 -> dist-capt2; footprint (none) -> Pin_Headers:Pin_Header_Straight_1x03_Pitch2.54mm
- P14: value CONN_01X03 -> dist-capt3; footprint (none) -> Pin_Headers:Pin_Header_Straight_1x03_Pitch2.54mm
- P15: value CONN_01X03 -> dist-capt6; footprint (none) -> Pin_Headers:Pin_Header_Straight_1x03_Pitch2.54mm

Commit message: fin PCB
Parts:
- renumbered P10 to P19, P11 to P20, P12 to P21, P13 to P22, P14 to P23, P15 to P24
Changed lines of the file:
@@
 EESchema Schematic File Version 2
+LIBS:carte-asser-1A-2016-2017-rescue
 LIBS:power
 LIBS:device
@@
 $Descr A4 11693 8268
 encoding utf-8
-Sheet 8 9
+Sheet 8 10
 Title ""
 Date ""
@@
 $EndDescr
 $Comp
-L +5V #PWR074
+L +5V #PWR072
 U 1 1 589FE6A9
 P 2400 1250
-F 0 "#PWR074" H 2400 1100 50  0001 C CNN
+F 0 "#PWR072" H 2400 1100 50  0001 C CNN
 F 1 "+5V" H 2400 1390 50  0000 C CNN
 F 2 "" H 2400 1250 50  0000 C CNN
@@
 	2400 2000 2400 2700
 $Comp
-L GND #PWR075
+L GND #PWR073
 U 1 1 589FE6CC
 P 2400 2700
-F 0 "#PWR075" H 2400 2450 50  0001 C CNN
+F 0 "#PWR073" H 2400 2450 50  0001 C CNN
 F 1 "GND" H 2400 2550 50  0000 C CNN
 F 2 "" H 2400 2700 50  0000 C CNN
@@
 c-distance6
 $Comp
-L +5V #PWR076
+L +5V #PWR074
 U 1 1 58A0A933
 P 5850 1250
-F 0 "#PWR076" H 5850 1100 50  0001 C CNN
+F 0 "#PWR074" H 5850 1100 50  0001 C CNN
 F 1 "+5V" H 5850 1390 50  0000 C CNN
 F 2 "" H 5850 1250 50  0000 C CNN
@@
 	5850 2000 5850 2700
 $Comp
-L GND #PWR077
+L GND #PWR075
 U 1 1 58A0A93C
 P 5850 2700
-F 0 "#PWR077" H 5850 2450 50  0001 C CNN
+F 0 "#PWR075" H 5850 2450 50  0001 C CNN
 F 1 "GND" H 5850 2550 50  0000 C CNN
 F 2 "" H 5850 2700 50  0000 C CNN
@@
 	4950 1200 4650 1200
 $Comp
-L CONN_01X03 P13
+L CONN_01X03 P22
 U 1 1 58A0A954
 P 6650 1900
-F 0 "P13" H 6650 2100 50  0000 C CNN
+F 0 "P22" H 6650 2100 50  0000 C CNN
 F 1 "dist-capt2" V 6750 1900 50  0000 C CNN
 F 2 "Pin_Headers:Pin_Header_Straight_1x03_Pitch2.54mm" H 6650 1900 50  0001 C CNN
@@
 $EndComp
 $Comp
-L +5V #PWR078
+L +5V #PWR076
 U 1 1 58A0AA92
 P 9150 1200
-F 0 "#PWR078" H 9150 1050 50  0001 C CNN
+F 0 "#PWR076" H 9150 1050 50  0001 C CNN
 F 1 "+5V" H 9150 1340 50  0000 C CNN
 F 2 "" H 9150 1200 50  0000 C CNN
@@
 	9150 1950 9150 2650
 $Comp
-L GND #PWR079
+L GND #PWR077
 U 1 1 58A0AA9B
 P 9150 2650
-F 0 "#PWR079" H 9150 2400 50  0001 C CNN
+F 0 "#PWR077" H 9150 2400 50  0001 C CNN
 F 1 "GND" H 9150 2500 50  0000 C CNN
 F 2 "" H 9150 2650 50  0000 C CNN
@@
 	8250 1150 7950 1150
 $Comp
-L CONN_01X03 P14
+L CONN_01X03 P23
 U 1 1 58A0AAB3
 P 9950 1850
-F 0 "P14" H 9950 2050 50  0000 C CNN
+F 0 "P23" H 9950 2050 50  0000 C CNN
 F 1 "dist-capt3" V 10050 1850 50  0000 C CNN
 F 2 "Pin_Headers:Pin_Header_Straight_1x03_Pitch2.54mm" H 9950 1850 50  0001 C CNN
@@
 $EndComp
 $Comp
-L +5V #PWR080
+L +5V #PWR078
 U 1 1 58A0AD2F
 P 9150 3950
-F 0 "#PWR080" H 9150 3800 50  0001 C CNN
+F 0 "#PWR078" H 9150 3800 50  0001 C CNN
 F 1 "+5V" H 9150 4090 50  0000 C CNN
 F 2 "" H 9150 3950 50  0000 C CNN
@@
 	9150 4700 9150 5400
 $Comp
-L GND #PWR081
+L GND #PWR079
 U 1 1 58A0AD38
 P 9150 5400
-F 0 "#PWR081" H 9150 5150 50  0001 C CNN
+F 0 "#PWR079" H 9150 5150 50  0001 C CNN
 F 1 "GND" H 9150 5250 50  0000 C CNN
 F 2 "" H 9150 5400 50  0000 C CNN
@@
 	8250 3900 7950 3900
 $Comp
-L CONN_01X03 P15
+L CONN_01X03 P24
 U 1 1 58A0AD50
 P 9950 4600
-F 0 "P15" H 9950 4800 50  0000 C CNN
+F 0 "P24" H 9950 4800 50  0000 C CNN
 F 1 "dist-capt6" V 10050 4600 50  0000 C CNN
 F 2 "Pin_Headers:Pin_Header_Straight_1x03_Pitch2.54mm" H 9950 4600 50  0001 C CNN
@@
 $EndComp
 $Comp
-L +5V #PWR082
+L +5V #PWR080
 U 1 1 58A0AEEE
 P 5800 4050
-F 0 "#PWR082" H 5800 3900 50  0001 C CNN
+F 0 "#PWR080" H 5800 3900 50  0001 C CNN
 F 1 "+5V" H 5800 4190 50  0000 C CNN
 F 2 "" H 5800 4050 50  0000 C CNN
@@
 	5800 4800 5800 5500
 $Comp
-L GND #PWR083
+L GND #PWR081
 U 1 1 58A0AEF7
 P 5800 5500
-F 0 "#PWR083" H 5800 5250 50  0001 C CNN
+F 0 "#PWR081" H 5800 5250 50  0001 C CNN
 F 1 "GND" H 5800 5350 50  0000 C CNN
 F 2 "" H 5800 5500 50  0000 C CNN
@@
 	4900 4000 4600 4000
 $Comp
-L CONN_01X03 P12
+L CONN_01X03 P21
 U 1 1 58A0AF0F
 P 6600 4700
-F 0 "P12" H 6600 4900 50  0000 C CNN
+F 0 "P21" H 6600 4900 50  0000 C CNN
 F 1 "dist-capt5" V 6700 4700 50  0000 C CNN
 F 2 "Pin_Headers:Pin_Header_Straight_1x03_Pitch2.54mm" H 6600 4700 50  0001 C CNN
@@
 $EndComp
 $Comp
-L +5V #PWR084
+L +5V #PWR082
 U 1 1 58A0B0DD
 P 2600 4250
-F 0 "#PWR084" H 2600 4100 50  0001 C CNN
+F 0 "#PWR082" H 2600 4100 50  0001 C CNN
 F 1 "+5V" H 2600 4390 50  0000 C CNN
 F 2 "" H 2600 4250 50  0000 C CNN
@@
 	2600 5000 2600 5700
 $Comp
-L GND #PWR085
+L GND #PWR083
 U 1 1 58A0B0E6
 P 2600 5700
-F 0 "#PWR085" H 2600 5450 50  0001 C CNN
+F 0 "#PWR083" H 2600 5450 50  0001 C CNN
 F 1 "GND" H 2600 5550 50  0000 C CNN
 F 2 "" H 2600 5700 50  0000 C CNN
@@
 	1700 4200 1400 4200
 $Comp
-L CONN_01X03 P11
+L CONN_01X03 P20
 U 1 1 58A0B0FE
 P 3400 4900
-F 0 "P11" H 3400 5100 50  0000 C CNN
+F 0 "P20" H 3400 5100 50  0000 C CNN
 F 1 "dist-capt4" V 3500 4900 50  0000 C CNN
 F 2 "Pin_Headers:Pin_Header_Straight_1x03_Pitch2.54mm" H 3400 4900 50  0001 C CNN
@@
 $EndComp
 $Comp
-L CONN_01X03 P10
+L CONN_01X03 P19
 U 1 1 58A09E89
 P 3200 1900
-F 0 "P10" H 3200 2100 50  0000 C CNN
+F 0 "P19" H 3200 2100 50  0000 C CNN
 F 1 "dist-capt1" V 3300 1900 50  0000 C CNN
 F 2 "Pin_Headers:Pin_Header_Straight_1x03_Pitch2.54mm" H 3200 1900 50  0001 C CNN
