File: carte-asser-1A-2016-2017/motor_cc_part.sch (KiCad schematic (older format))
At the start: 8 parts

Commit message: Fin PCB
Parts:
- removed D? (x2): D_Small, symbol D_Small
- gave numbers to parts that had none: 6
Connections:
- net at D1.2 (A), D3.1 (K), H1.3 (born1_motor1): now also P9.1 (P1)
- net at D2.2 (A), D4.1 (K), H1.6 (born2_motor1): now also P9.2 (P2)
- net active-cc renamed enable-cc
Changed lines of the file:
@@
 LIBS:valves
 LIBS:robot_1A
-LIBS:carte-asser-1A-cache
 LIBS:carte-asser-1A-2016-2017-cache
 EELAYER 25 0
@@
 $Descr A4 11693 8268
 encoding utf-8
-Sheet 3 7
+Sheet 3 8
 Title ""
 Date ""
@@
 $EndDescr
 $Comp
-L H-bridge H?
+L H-bridge H1
 U 1 1 58937B34
 P 5800 4250
-F 0 "H?" H 6950 4550 60  0000 C CNN
+F 0 "H1" H 6950 4550 60  0000 C CNN
 F 1 "H-bridge" H 7000 4950 60  0000 C CNN
 F 2 "" H 8150 6350 60  0001 C CNN
@@
 	5750 3900 5950 3900
 $Comp
-L GND #PWR019
+L GND #PWR020
 U 1 1 58937BDB
 P 5750 3900
-F 0 "#PWR019" H 5750 3650 50  0001 C CNN
+F 0 "#PWR020" H 5750 3650 50  0001 C CNN
 F 1 "GND" H 5750 3750 50  0000 C CNN
 F 2 "" H 5750 3900 50  0000 C CNN
@@
 	5600 4200 5600 4850
 Text HLabel 5800 3100 1    60   Input ~ 0
-active-cc
+enable-cc
 Text HLabel 5450 3100 1    60   Input ~ 0
 speed-cc
@@
 	5500 4100 5950 4100
 $Comp
-L GND #PWR020
+L GND #PWR021
 U 1 1 58937FA4
 P 3600 3550
-F 0 "#PWR020" H 3600 3300 50  0001 C CNN
+F 0 "#PWR021" H 3600 3300 50  0001 C CNN
 F 1 "GND" H 3600 3400 50  0000 C CNN
 F 2 "" H 3600 3550 50  0000 C CNN
@@
 Connection ~ 2550 3850
 $Comp
-L CONN_01X02 P?
+L CONN_01X02 P9
 U 1 1 589380DD
 P 3250 3550
-F 0 "P?" H 3250 3700 50  0000 C CNN
+F 0 "P9" H 3250 3700 50  0000 C CNN
 F 1 "CONN_01X02" V 3350 3550 50  0000 C CNN
 F 2 "" H 3250 3550 50  0000 C CNN
@@
 $EndComp
 $Comp
-L D_Schottky D?
+L D_Schottky D3
 U 1 1 5893F78D
 P 3350 3300
-F 0 "D?" H 3350 3400 50  0000 C CNN
+F 0 "D3" H 3350 3400 50  0000 C CNN
 F 1 "D_Schottky" H 3350 3200 50  0000 C CNN
 F 2 "" H 3350 3300 50  0000 C CNN
@@
 $EndComp
 $Comp
-L D_Schottky D?
+L D_Schottky D1
 U 1 1 5893F7B2
 P 2700 3300
-F 0 "D?" H 2700 3400 50  0000 C CNN
+F 0 "D1" H 2700 3400 50  0000 C CNN
 F 1 "D_Schottky" H 2700 3200 50  0000 C CNN
 F 2 "" H 2700 3300 50  0000 C CNN
@@
 $EndComp
 $Comp
-L D_Schottky D?
+L D_Schottky D2
 U 1 1 5893F7CF
 P 2700 3850
-F 0 "D?" H 2700 3950 50  0000 C CNN
+F 0 "D2" H 2700 3950 50  0000 C CNN
 F 1 "D_Schottky" H 2700 3750 50  0000 C CNN
 F 2 "" H 2700 3850 50  0000 C CNN
@@
 $EndComp
 $Comp
-L D_Schottky D?
+L D_Schottky D4
 U 1 1 5893F7EE
 P 3350 3850
-F 0 "D?" H 3350 3950 50  0000 C CNN
+F 0 "D4" H 3350 3950 50  0000 C CNN
 F 1 "D_Schottky" H 3350 3750 50  0000 C CNN
 F 2 "" H 3350 3850 50  0000 C CNN
@@
 	1    0    0    -1
 $EndComp
-$Comp
-L D_Small D?
-U 1 1 589CF9DB
-P 3050 3400
-F 0 "D?" H 3000 3480 50  0000 L CNN
-F 1 "D_Small" H 2900 3320 50  0000 L CNN
-F 2 "" V 3050 3400 50  0000 C CNN
-F 3 "" V 3050 3400 50  0000 C CNN
-	1    3050 3400
-	0    -1   -1   0
-$EndComp
-$Comp
-L D_Small D?
-U 1 1 589CFA04
-P 3050 3700
-F 0 "D?" H 3000 3780 50  0000 L CNN
-F 1 "D_Small" H 2900 3620 50  0000 L CNN
-F 2 "" V 3050 3700 50  0000 C CNN
-F 3 "" V 3050 3700 50  0000 C CNN
-	1    3050 3700
-	0    1    1    0
-$EndComp
 Wire Wire Line
-	3050 3800 3050 4000
-Wire Wire Line
-	3050 3150 3050 3300
+	3050 3150 3050 3500
 Wire Wire Line
 	5600 4850 5950 4850
@@
 	5950 4850 5950 4750
 $Comp
-L +8V #PWR021
+L +8V #PWR022
 U 1 1 589D6B4D
 P 5950 4750
-F 0 "#PWR021" H 5950 4600 50  0001 C CNN
+F 0 "#PWR022" H 5950 4600 50  0001 C CNN
 F 1 "+8V" H 5950 4890 50  0000 C CNN
 F 2 "" H 5950 4750 50  0000 C CNN
@@
 	1    0    0    -1
 $EndComp
+Wire Wire Line
+	3050 3600 3050 4000
 $EndSCHEMATC

Commit message: PCB
Parts:
- D1, D2, D3, D4: footprint (none) -> Discret:R4-LARGE_PADS
- H1: footprint (none) -> Housings_DIP:DIP-16_W7.62mm
- P9: value CONN_01X02 -> cc-motor; footprint (none) -> Pin_Headers:Pin_Header_Straight_1x02_Pitch2.54mm
Changed lines of the file:
@@
 $Descr A4 11693 8268
 encoding utf-8
-Sheet 3 8
+Sheet 3 9
 Title ""
 Date ""
@@
 F 0 "H1" H 6950 4550 60  0000 C CNN
 F 1 "H-bridge" H 7000 4950 60  0000 C CNN
-F 2 "" H 8150 6350 60  0001 C CNN
+F 2 "Housings_DIP:DIP-16_W7.62mm" H 8150 6350 60  0001 C CNN
 F 3 "" H 8150 6350 60  0001 C CNN
 	1    5800 4250
@@
 P 3250 3550
 F 0 "P9" H 3250 3700 50  0000 C CNN
-F 1 "CONN_01X02" V 3350 3550 50  0000 C CNN
-F 2 "" H 3250 3550 50  0000 C CNN
+F 1 "cc-motor" V 3350 3550 50  0000 C CNN
+F 2 "Pin_Headers:Pin_Header_Straight_1x02_Pitch2.54mm" H 3250 3550 50  0001 C CNN
 F 3 "" H 3250 3550 50  0000 C CNN
 	1    3250 3550
@@
 F 0 "D3" H 3350 3400 50  0000 C CNN
 F 1 "D_Schottky" H 3350 3200 50  0000 C CNN
-F 2 "" H 3350 3300 50  0000 C CNN
+F 2 "Discret:R4-LARGE_PADS" H 3350 3300 50  0001 C CNN
 F 3 "" H 3350 3300 50  0000 C CNN
 	1    3350 3300
@@
 F 0 "D1" H 2700 3400 50  0000 C CNN
 F 1 "D_Schottky" H 2700 3200 50  0000 C CNN
-F 2 "" H 2700 3300 50  0000 C CNN
+F 2 "Discret:R4-LARGE_PADS" H 2700 3300 50  0001 C CNN
 F 3 "" H 2700 3300 50  0000 C CNN
 	1    2700 3300
@@
 F 0 "D2" H 2700 3950 50  0000 C CNN
 F 1 "D_Schottky" H 2700 3750 50  0000 C CNN
-F 2 "" H 2700 3850 50  0000 C CNN
+F 2 "Discret:R4-LARGE_PADS" H 2700 3850 50  0001 C CNN
 F 3 "" H 2700 3850 50  0000 C CNN
 	1    2700 3850
@@
 F 0 "D4" H 3350 3950 50  0000 C CNN
 F 1 "D_Schottky" H 3350 3750 50  0000 C CNN
-F 2 "" H 3350 3850 50  0000 C CNN
+F 2 "Discret:R4-LARGE_PADS" H 3350 3850 50  0001 C CNN
 F 3 "" H 3350 3850 50  0000 C CNN
 	1    3350 3850

Commit message: fin PCB
Parts:
- renumbered P9 to P8
Connections:
- no-connect marks 0 -> 8
Changed lines of the file:
@@
 EESchema Schematic File Version 2
+LIBS:carte-asser-1A-2016-2017-rescue
 LIBS:power
 LIBS:device
@@
 $Descr A4 11693 8268
 encoding utf-8
-Sheet 3 9
+Sheet 3 10
 Title ""
 Date ""
@@
 Comment4 ""
 $EndDescr
-$Comp
-L H-bridge H1
-U 1 1 58937B34
-P 5800 4250
-F 0 "H1" H 6950 4550 60  0000 C CNN
-F 1 "H-bridge" H 7000 4950 60  0000 C CNN
-F 2 "Housings_DIP:DIP-16_W7.62mm" H 8150 6350 60  0001 C CNN
-F 3 "" H 8150 6350 60  0001 C CNN
-	1    5800 4250
-	1    0    0    -1
-$EndComp
 Wire Wire Line
 	5950 3500 5800 3500
@@
 Connection ~ 2550 3850
 $Comp
-L CONN_01X02 P9
+L CONN_01X02 P8
 U 1 1 589380DD
 P 3250 3550
-F 0 "P9" H 3250 3700 50  0000 C CNN
+F 0 "P8" H 3250 3700 50  0000 C CNN
 F 1 "cc-motor" V 3350 3550 50  0000 C CNN
 F 2 "Pin_Headers:Pin_Header_Straight_1x02_Pitch2.54mm" H 3250 3550 50  0001 C CNN
@@
 Wire Wire Line
 	3050 3600 3050 4000
+$Comp
+L H-bridge H1
+U 1 1 58D7D568
+P 5800 4250
+F 0 "H1" H 6950 4550 60  0000 C CNN
+F 1 "H-bridge" H 7000 4950 60  0000 C CNN
+F 2 "Housings_DIP:DIP-16_W7.62mm" H 8150 6350 60  0001 C CNN
+F 3 "" H 8150 6350 60  0001 C CNN
+	1    5800 4250
+	1    0    0    -1
+$EndComp
+NoConn ~ 8100 3500
+NoConn ~ 8100 3600
+NoConn ~ 8100 3700
+NoConn ~ 8100 3800
+NoConn ~ 8100 3900
+NoConn ~ 8100 4000
+NoConn ~ 8100 4100
+NoConn ~ 8100 4200
 $EndSCHEMATC
