File: carte-asser-1A-2016-2017/pwr_part.sch (KiCad schematic (older format))
At the start: 16 parts

Commit message: Fin PCB
Parts:
- removed D?: D_Small, symbol D_Small
- added D7: D_Schottky, symbol D_Schottky
- added F1: FUSE, symbol FUSE
- C5: renamed from C?; value C -> 100µ
- C6, C7: renamed from C?; value C -> 1µ
- R1: renamed from R?; value R -> 300
- R2: renamed from R?; value R -> 1.3k
- R3: renamed from R?; value R -> 500
- gave numbers to parts that had none: 9
Connections:
- net +15V: now also D7.1 (K), F1.1
- net GND: now also U6.1 (GND), D7.2 (A)
- net at U7.1: now also F1.2
Other:
- moved on the sheet: D8, R2

Commit message: PCB
Parts:
- C5, C6, C7: footprint (none) -> Capacitors_ThroughHole:C_Rect_L7.0mm_W2.5mm_P5.00mm
- D10, D5, D6, D7, D8, D9, F1, R1, R2, R3: footprint (none) -> Discret:R4-LARGE_PADS
- U5: value B_Plug_5mm -> +5V; footprint (none) -> B plug:B plug 5mm
- U6: footprint (none) -> TO_SOT_Packages_SMD:SOT89-3_Housing
- U7: value B_Plug_5mm -> +15V; footprint (none) -> B plug:B plug 5mm
- U8: value B_Plug_5mm -> +7.3V; footprint (none) -> B plug:B plug 5mm
Changed lines of the file:
@@
 $Descr A4 11693 8268
 encoding utf-8
-Sheet 4 8
+Sheet 4 9
 Title ""
 Date ""
@@
 P 1250 1050
 F 0 "U5" H 1250 1450 60  0000 C CNN
-F 1 "B_Plug_5mm" H 1250 1550 60  0000 C CNN
-F 2 "" H 1250 1050 60  0000 C CNN
+F 1 "+5V" H 1250 1550 60  0000 C CNN
+F 2 "B plug:B plug 5mm" H 1250 1050 60  0001 C CNN
 F 3 "" H 1250 1050 60  0000 C CNN
 	1    1250 1050
@@
 F 0 "D5" V 1250 1530 50  0000 L CNN
 F 1 "D_Small" H 1150 1370 50  0000 L CNN
-F 2 "" V 1300 1450 50  0000 C CNN
+F 2 "Discret:R4-LARGE_PADS" V 1300 1450 50  0001 C CNN
 F 3 "" V 1300 1450 50  0000 C CNN
 	1    1300 1450
@@
 F 0 "U6" H 2650 3450 50  0000 C CNN
 F 1 "MCP1702" H 2550 3950 50  0000 C CNN
-F 2 "" H 2550 3700 50  0000 C CNN
+F 2 "TO_SOT_Packages_SMD:SOT89-3_Housing" H 2550 3700 50  0001 C CNN
 F 3 "" H 2550 3700 50  0000 C CNN
 	1    2550 3700
@@
 F 0 "C6" H 1775 4250 50  0000 L CNN
 F 1 "1µ" H 1775 4050 50  0000 L CNN
-F 2 "" H 1788 4000 50  0000 C CNN
+F 2 "Capacitors_ThroughHole:C_Rect_L7.0mm_W2.5mm_P5.00mm" H 1788 4000 50  0001 C CNN
 F 3 "" H 1750 4150 50  0000 C CNN
 	1    1750 4150
@@
 F 0 "C5" H 1325 4250 50  0000 L CNN
 F 1 "100µ" H 1325 4050 50  0000 L CNN
-F 2 "" H 1338 4000 50  0000 C CNN
+F 2 "Capacitors_ThroughHole:C_Rect_L7.0mm_W2.5mm_P5.00mm" H 1338 4000 50  0001 C CNN
 F 3 "" H 1300 4150 50  0000 C CNN
 	1    1300 4150
@@
 F 0 "C7" H 3325 4250 50  0000 L CNN
 F 1 "1µ" H 3325 4050 50  0000 L CNN
-F 2 "" H 3338 4000 50  0000 C CNN
+F 2 "Capacitors_ThroughHole:C_Rect_L7.0mm_W2.5mm_P5.00mm" H 3338 4000 50  0001 C CNN
 F 3 "" H 3300 4150 50  0000 C CNN
 	1    3300 4150
@@
 F 0 "D6" H 1600 2150 50  0000 C CNN
 F 1 "LED" H 1600 1950 50  0000 C CNN
-F 2 "" H 1600 2050 50  0000 C CNN
+F 2 "Discret:R4-LARGE_PADS" H 1600 2050 50  0001 C CNN
 F 3 "" H 1600 2050 50  0000 C CNN
 	1    1600 2050
@@
 F 0 "R1" V 2230 2050 50  0000 C CNN
 F 1 "300" V 2150 2050 50  0000 C CNN
-F 2 "" V 2080 2050 50  0000 C CNN
+F 2 "Discret:R4-LARGE_PADS" V 2080 2050 50  0001 C CNN
 F 3 "" H 2150 2050 50  0000 C CNN
 	1    2150 2050
@@
 P 4000 1150
 F 0 "U7" H 3900 1000 60  0000 C CNN
-F 1 "B_Plug_5mm" V 3650 1150 60  0000 C CNN
-F 2 "" H 4000 1150 60  0000 C CNN
+F 1 "+15V" V 3650 1150 60  0000 C CNN
+F 2 "B plug:B plug 5mm" H 4000 1150 60  0001 C CNN
 F 3 "" H 4000 1150 60  0000 C CNN
 	1    4000 1150
@@
 F 0 "D8" H 4250 2500 50  0000 C CNN
 F 1 "LED" H 4250 2300 50  0000 C CNN
-F 2 "" H 4250 2400 50  0000 C CNN
+F 2 "Discret:R4-LARGE_PADS" H 4250 2400 50  0001 C CNN
 F 3 "" H 4250 2400 50  0000 C CNN
 	1    4250 2400
@@
 F 0 "R2" V 4880 2400 50  0000 C CNN
 F 1 "1.3k" V 4800 2400 50  0000 C CNN
-F 2 "" V 4730 2400 50  0000 C CNN
+F 2 "Discret:R4-LARGE_PADS" V 4730 2400 50  0001 C CNN
 F 3 "" H 4800 2400 50  0000 C CNN
 	1    4800 2400
@@
 P 6900 1200
 F 0 "U8" H 6900 1600 60  0000 C CNN
-F 1 "B_Plug_5mm" H 6900 1700 60  0000 C CNN
-F 2 "" H 6900 1200 60  0000 C CNN
+F 1 "+7.3V" H 6900 1700 60  0000 C CNN
+F 2 "B plug:B plug 5mm" H 6900 1200 60  0001 C CNN
 F 3 "" H 6900 1200 60  0000 C CNN
 	1    6900 1200
@@
 F 0 "D9" V 6900 1680 50  0000 L CNN
 F 1 "D_Small" H 6800 1520 50  0000 L CNN
-F 2 "" V 6950 1600 50  0000 C CNN
+F 2 "Discret:R4-LARGE_PADS" V 6950 1600 50  0001 C CNN
 F 3 "" V 6950 1600 50  0000 C CNN
 	1    6950 1600
@@
 F 0 "D10" H 7250 2300 50  0000 C CNN
 F 1 "LED" H 7250 2100 50  0000 C CNN
-F 2 "" H 7250 2200 50  0000 C CNN
+F 2 "Discret:R4-LARGE_PADS" H 7250 2200 50  0001 C CNN
 F 3 "" H 7250 2200 50  0000 C CNN
 	1    7250 2200
@@
 F 0 "R3" V 7880 2200 50  0000 C CNN
 F 1 "500" V 7800 2200 50  0000 C CNN
-F 2 "" V 7730 2200 50  0000 C CNN
+F 2 "Discret:R4-LARGE_PADS" V 7730 2200 50  0001 C CNN
 F 3 "" H 7800 2200 50  0000 C CNN
 	1    7800 2200
@@
 F 0 "F1" H 4150 1650 50  0000 C CNN
 F 1 "FUSE" H 3950 1550 50  0000 C CNN
-F 2 "" H 4050 1600 50  0000 C CNN
+F 2 "Discret:R4-LARGE_PADS" H 4050 1600 50  0001 C CNN
 F 3 "" H 4050 1600 50  0000 C CNN
 	1    4050 1600
@@
 F 0 "D7" H 3850 2050 50  0000 C CNN
 F 1 "D_Schottky" H 3850 1850 50  0000 C CNN
-F 2 "" H 3850 1950 50  0000 C CNN
+F 2 "Discret:R4-LARGE_PADS" H 3850 1950 50  0001 C CNN
 F 3 "" H 3850 1950 50  0000 C CNN
 	1    3850 1950

Commit message: fin PCB
Parts:
- removed C5: 100µ, Capacitors_ThroughHole:C_Rect_L7.0mm_W2.5mm_P5.00mm, symbol C
- removed C6, C7: 1µ, Capacitors_ThroughHole:C_Rect_L7.0mm_W2.5mm_P5.00mm, symbol C
- removed U6: MCP1702, TO_SOT_Packages_SMD:SOT89-3_Housing, symbol MCP1702
- added R18: 270, Discret:R4-LARGE_PADS, symbol R
- added R19: 330, Discret:R4-LARGE_PADS, symbol R
- F1: footprint Discret:R4-LARGE_PADS -> Resistors_SMD:R_2816_HandSoldering
- renumbered R1 to R2, R2 to R3, R3 to R4
Connections:
- net +3V3: now also R18.2, R19.1
- net +5V: now also R18.1
- net GND: now also R19.2
Changed lines of the file:
@@
 EESchema Schematic File Version 2
+LIBS:carte-asser-1A-2016-2017-rescue
 LIBS:power
 LIBS:device
@@
 $Descr A4 11693 8268
 encoding utf-8
-Sheet 4 9
+Sheet 4 10
 Title ""
 Date ""
@@
 $EndComp
 $Comp
-L MCP1702 U6
-U 1 1 589C7316
-P 2550 3700
-F 0 "U6" H 2650 3450 50  0000 C CNN
-F 1 "MCP1702" H 2550 3950 50  0000 C CNN
-F 2 "TO_SOT_Packages_SMD:SOT89-3_Housing" H 2550 3700 50  0001 C CNN
-F 3 "" H 2550 3700 50  0000 C CNN
-	1    2550 3700
-	1    0    0    -1
-$EndComp
-$Comp
-L C C6
-U 1 1 589C7354
-P 1750 4150
-F 0 "C6" H 1775 4250 50  0000 L CNN
-F 1 "1µ" H 1775 4050 50  0000 L CNN
-F 2 "Capacitors_ThroughHole:C_Rect_L7.0mm_W2.5mm_P5.00mm" H 1788 4000 50  0001 C CNN
-F 3 "" H 1750 4150 50  0000 C CNN
-	1    1750 4150
-	1    0    0    -1
-$EndComp
-$Comp
-L C C5
-U 1 1 589C73E9
-P 1300 4150
-F 0 "C5" H 1325 4250 50  0000 L CNN
-F 1 "100µ" H 1325 4050 50  0000 L CNN
-F 2 "Capacitors_ThroughHole:C_Rect_L7.0mm_W2.5mm_P5.00mm" H 1338 4000 50  0001 C CNN
-F 3 "" H 1300 4150 50  0000 C CNN
-	1    1300 4150
-	1    0    0    -1
-$EndComp
-$Comp
-L +5V #PWR025
-U 1 1 589C7408
-P 1750 3400
-F 0 "#PWR025" H 1750 3250 50  0001 C CNN
-F 1 "+5V" H 1750 3540 50  0000 C CNN
-F 2 "" H 1750 3400 50  0000 C CNN
-F 3 "" H 1750 3400 50  0000 C CNN
-	1    1750 3400
-	1    0    0    -1
-$EndComp
-$Comp
-L +3.3V #PWR026
-U 1 1 589C7453
-P 3300 3400
-F 0 "#PWR026" H 3300 3250 50  0001 C CNN
-F 1 "+3.3V" H 3300 3540 50  0000 C CNN
-F 2 "" H 3300 3400 50  0000 C CNN
-F 3 "" H 3300 3400 50  0000 C CNN
-	1    3300 3400
-	1    0    0    -1
-$EndComp
-$Comp
-L C C7
-U 1 1 589C7471
-P 3300 4150
-F 0 "C7" H 3325 4250 50  0000 L CNN
-F 1 "1µ" H 3325 4050 50  0000 L CNN
-F 2 "Capacitors_ThroughHole:C_Rect_L7.0mm_W2.5mm_P5.00mm" H 3338 4000 50  0001 C CNN
-F 3 "" H 3300 4150 50  0000 C CNN
-	1    3300 4150
-	1    0    0    -1
-$EndComp
-$Comp
-L GND #PWR027
-U 1 1 589C760B
-P 3300 4450
-F 0 "#PWR027" H 3300 4200 50  0001 C CNN
-F 1 "GND" H 3300 4300 50  0000 C CNN
-F 2 "" H 3300 4450 50  0000 C CNN
-F 3 "" H 3300 4450 50  0000 C CNN
-	1    3300 4450
-	1    0    0    -1
-$EndComp
-$Comp
-L GND #PWR028
-U 1 1 589C762B
-P 1750 4450
-F 0 "#PWR028" H 1750 4200 50  0001 C CNN
-F 1 "GND" H 1750 4300 50  0000 C CNN
-F 2 "" H 1750 4450 50  0000 C CNN
-F 3 "" H 1750 4450 50  0000 C CNN
-	1    1750 4450
-	1    0    0    -1
-$EndComp
-$Comp
-L GND #PWR029
-U 1 1 589C764B
-P 1300 4450
-F 0 "#PWR029" H 1300 4200 50  0001 C CNN
-F 1 "GND" H 1300 4300 50  0000 C CNN
-F 2 "" H 1300 4450 50  0000 C CNN
-F 3 "" H 1300 4450 50  0000 C CNN
-	1    1300 4450
-	1    0    0    -1
-$EndComp
-$Comp
-L PWR_FLAG #FLG030
+L PWR_FLAG #FLG025
 U 1 1 589C91A5
 P 1000 2100
-F 0 "#FLG030" H 1000 2195 50  0001 C CNN
+F 0 "#FLG025" H 1000 2195 50  0001 C CNN
 F 1 "PWR_FLAG" H 1000 2280 50  0000 C CNN
 F 2 "" H 1000 2100 50  0000 C CNN
@@
 $EndComp
 $Comp
-L R R1
+L R R2
 U 1 1 589C92BD
 P 2150 2050
-F 0 "R1" V 2230 2050 50  0000 C CNN
+F 0 "R2" V 2230 2050 50  0000 C CNN
 F 1 "300" V 2150 2050 50  0000 C CNN
 F 2 "Discret:R4-LARGE_PADS" V 2080 2050 50  0001 C CNN
@@
 $EndComp
 $Comp
-L GND #PWR031
+L GND #PWR026
 U 1 1 589C94A5
 P 2500 2150
-F 0 "#PWR031" H 2500 1900 50  0001 C CNN
+F 0 "#PWR026" H 2500 1900 50  0001 C CNN
 F 1 "GND" H 2500 2000 50  0000 C CNN
 F 2 "" H 2500 2150 50  0000 C CNN
@@
 $EndComp
 $Comp
-L PWR_FLAG #FLG032
+L PWR_FLAG #FLG027
 U 1 1 589C9645
 P 900 1150
-F 0 "#FLG032" H 900 1245 50  0001 C CNN
+F 0 "#FLG027" H 900 1245 50  0001 C CNN
 F 1 "PWR_FLAG" H 900 1330 50  0000 C CNN
 F 2 "" H 900 1150 50  0000 C CNN
@@
 $EndComp
 $Comp
-L PWR_FLAG #FLG033
+L PWR_FLAG #FLG028
 U 1 1 589CBE99
 P 3750 2550
-F 0 "#FLG033" H 3750 2645 50  0001 C CNN
+F 0 "#FLG028" H 3750 2645 50  0001 C CNN
 F 1 "PWR_FLAG" H 3750 2730 50  0000 C CNN
 F 2 "" H 3750 2550 50  0000 C CNN
@@
 $EndComp
 $Comp
-L R R2
+L R R3
 U 1 1 589CBEA5
 P 4800 2400
-F 0 "R2" V 4880 2400 50  0000 C CNN
+F 0 "R3" V 4880 2400 50  0000 C CNN
 F 1 "1.3k" V 4800 2400 50  0000 C CNN
 F 2 "Discret:R4-LARGE_PADS" V 4730 2400 50  0001 C CNN
@@
 $EndComp
 $Comp
-L GND #PWR034
+L GND #PWR029
 U 1 1 589CBEAB
 P 5150 2500
-F 0 "#PWR034" H 5150 2250 50  0001 C CNN
+F 0 "#PWR029" H 5150 2250 50  0001 C CNN
 F 1 "GND" H 5150 2350 50  0000 C CNN
 F 2 "" H 5150 2500 50  0000 C CNN
@@
 $EndComp
 $Comp
-L GND #PWR035
+L GND #PWR030
 U 1 1 589CC007
 P 6550 1500
-F 0 "#PWR035" H 6550 1250 50  0001 C CNN
+F 0 "#PWR030" H 6550 1250 50  0001 C CNN
 F 1 "GND" H 6550 1350 50  0000 C CNN
 F 2 "" H 6550 1500 50  0000 C CNN
@@
 $EndComp
 $Comp
-L PWR_FLAG #FLG036
+L PWR_FLAG #FLG031
 U 1 1 589CC00D
 P 6650 2250
-F 0 "#FLG036" H 6650 2345 50  0001 C CNN
+F 0 "#FLG031" H 6650 2345 50  0001 C CNN
 F 1 "PWR_FLAG" H 6650 2430 50  0000 C CNN
 F 2 "" H 6650 2250 50  0000 C CNN
@@
 $EndComp
 $Comp
-L R R3
+L R R4
 U 1 1 589CC019
 P 7800 2200
-F 0 "R3" V 7880 2200 50  0000 C CNN
+F 0 "R4" V 7880 2200 50  0000 C CNN
 F 1 "500" V 7800 2200 50  0000 C CNN
 F 2 "Discret:R4-LARGE_PADS" V 7730 2200 50  0001 C CNN
@@
 $EndComp
 $Comp
-L GND #PWR037
+L GND #PWR032
 U 1 1 589CC01F
 P 8150 2300
-F 0 "#PWR037" H 8150 2050 50  0001 C CNN
+F 0 "#PWR032" H 8150 2050 50  0001 C CNN
 F 1 "GND" H 8150 2150 50  0000 C CNN
 F 2 "" H 8150 2300 50  0000 C CNN
@@
 $EndComp
 $Comp
-L +15V #PWR038
+L +15V #PWR033
 U 1 1 589CC0EC
 P 3750 2300
-F 0 "#PWR038" H 3750 2150 50  0001 C CNN
+F 0 "#PWR033" H 3750 2150 50  0001 C CNN
 F 1 "+15V" H 3750 2440 50  0000 C CNN
 F 2 "" H 3750 2300 50  0000 C CNN
@@
 $EndComp
 $Comp
-L +8V #PWR039
+L +8V #PWR034
 U 1 1 589CC1A1
 P 6650 2000
-F 0 "#PWR039" H 6650 1850 50  0001 C CNN
+F 0 "#PWR034" H 6650 1850 50  0001 C CNN
 F 1 "+8V" H 6650 2140 50  0000 C CNN
 F 2 "" H 6650 2000 50  0000 C CNN
 F 3 "" H 6650 2000 50  0000 C CNN
 	1    6650 2000
-	1    0    0    -1
-$EndComp
-$Comp
-L GND #PWR040
-U 1 1 58A70768
-P 2550 4200
-F 0 "#PWR040" H 2550 3950 50  0001 C CNN
-F 1 "GND" H 2550 4050 50  0000 C CNN
-F 2 "" H 2550 4200 50  0000 C CNN
-F 3 "" H 2550 4200 50  0000 C CNN
-	1    2550 4200
 	1    0    0    -1
 $EndComp
@@
 F 0 "F1" H 4150 1650 50  0000 C CNN
 F 1 "FUSE" H 3950 1550 50  0000 C CNN
-F 2 "Discret:R4-LARGE_PADS" H 4050 1600 50  0001 C CNN
+F 2 "Resistors_SMD:R_2816_HandSoldering" H 4050 1600 50  0001 C CNN
 F 3 "" H 4050 1600 50  0000 C CNN
 	1    4050 1600
@@
 $EndComp
 $Comp
-L GND #PWR041
+L GND #PWR035
 U 1 1 58AB25F6
 P 3300 1450
-F 0 "#PWR041" H 3300 1200 50  0001 C CNN
+F 0 "#PWR035" H 3300 1200 50  0001 C CNN
 F 1 "GND" H 3300 1300 50  0000 C CNN
 F 2 "" H 3300 1450 50  0000 C CNN
@@
 $EndComp
 Wire Wire Line
-	2200 3650 1300 3650
-Wire Wire Line
-	1300 3650 1300 4000
-Wire Wire Line
-	1750 3400 1750 4000
-Connection ~ 1750 3650
-Wire Wire Line
-	2900 3650 3300 3650
-Wire Wire Line
-	3300 3400 3300 4000
-Connection ~ 3300 3650
-Wire Wire Line
-	3300 4300 3300 4450
-Wire Wire Line
-	1750 4300 1750 4450
-Wire Wire Line
-	1300 4300 1300 4450
-Wire Wire Line
 	1200 1150 1200 1250
 Wire Wire Line
@@
 Wire Wire Line
 	8150 2200 8150 2300
-Connection ~ 3300 4400
-Wire Wire Line
-	2550 4000 2550 4200
 Wire Wire Line
 	4050 1250 4050 1350
@@
 Connection ~ 4050 1300
 $Comp
-L PWR_FLAG #FLG042
+L PWR_FLAG #FLG036
 U 1 1 58AFD01A
 P 4400 1150
-F 0 "#FLG042" H 4400 1245 50  0001 C CNN
+F 0 "#FLG036" H 4400 1245 50  0001 C CNN
 F 1 "PWR_FLAG" H 4400 1330 50  0000 C CNN
 F 2 "" H 4400 1150 50  0000 C CNN
@@
 Wire Wire Line
 	4400 1300 4400 1150
+$Comp
+L +5V #PWR037
+U 1 1 58D7FFB3
+P 2800 3900
+F 0 "#PWR037" H 2800 3750 50  0001 C CNN
+F 1 "+5V" H 2800 4040 50  0000 C CNN
+F 2 "" H 2800 3900 50  0000 C CNN
+F 3 "" H 2800 3900 50  0000 C CNN
+	1    2800 3900
+	1    0    0    -1
+$EndComp
+$Comp
+L R R18
+U 1 1 58D7FFE1
+P 2800 4300
+F 0 "R18" V 2880 4300 50  0000 C CNN
+F 1 "270" V 2800 4300 50  0000 C CNN
+F 2 "Discret:R4-LARGE_PADS" V 2730 4300 50  0001 C CNN
+F 3 "" H 2800 4300 50  0000 C CNN
+	1    2800 4300
+	1    0    0    -1
+$EndComp
+$Comp
+L R R19
+U 1 1 58D80052
+P 2800 4900
+F 0 "R19" V 2880 4900 50  0000 C CNN
+F 1 "330" V 2800 4900 50  0000 C CNN
+F 2 "Discret:R4-LARGE_PADS" V 2730 4900 50  0001 C CNN
+F 3 "" H 2800 4900 50  0000 C CNN
+	1    2800 4900
+	1    0    0    -1
+$EndComp
+$Comp
+L GND #PWR038
+U 1 1 58D8030C
+P 2800 5400
+F 0 "#PWR038" H 2800 5150 50  0001 C CNN
+F 1 "GND" H 2800 5250 50  0000 C CNN
+F 2 "" H 2800 5400 50  0000 C CNN
+F 3 "" H 2800 5400 50  0000 C CNN
+	1    2800 5400
+	1    0    0    -1
+$EndComp
+$Comp
+L +3.3V #PWR039
+U 1 1 58D8033E
+P 4000 4450
+F 0 "#PWR039" H 4000 4300 50  0001 C CNN
+F 1 "+3.3V" H 4000 4590 50  0000 C CNN
+F 2 "" H 4000 4450 50  0000 C CNN
+F 3 "" H 4000 4450 50  0000 C CNN
+	1    4000 4450
+	1    0    0    -1
+$EndComp
+Wire Wire Line
+	2800 3900 2800 4150
+Wire Wire Line
+	2800 4450 2800 4750
+Wire Wire Line
+	4000 4450 4000 4550
+Wire Wire Line
+	2800 4550 4350 4550
+Connection ~ 2800 4550
+Wire Wire Line
+	2800 5050 2800 5400
+Wire Wire Line
+	4350 4550 4350 4450
+Connection ~ 4000 4550
+$Comp
+L PWR_FLAG #FLG040
+U 1 1 58D81335
+P 4350 4450
+F 0 "#FLG040" H 4350 4545 50  0001 C CNN
+F 1 "PWR_FLAG" H 4350 4630 50  0000 C CNN
+F 2 "" H 4350 4450 50  0000 C CNN
+F 3 "" H 4350 4450 50  0000 C CNN
+	1    4350 4450
+	1    0    0    -1
+$EndComp
 $EndSCHEMATC
