File: carte-asser-1A-2016-2017/stepstick_part.sch (KiCad schematic (older format))
At the start: 28 parts

Commit message: Fin PCB
Parts:
- removed D? (x16): D_Small, symbol D_Small
- C1, C2, C3, C4: renamed from C?; value C -> 100µ
- gave numbers to parts that had none: 8
Connections:
- net +15V: now also C1.1, C2.1, C3.1, C4.1
- net GND: now also C1.2, C2.2, C3.2, C4.2
- net at P5.1 (P1): now also U1.~ (VMOT)
- net at P5.2 (P2): now also U1.~ (VMOT)
- net at P5.3 (P3): now also U1.~ (VMOT)
- net at P5.4 (P4): now also U1.~ (VMOT)
- net at P6.1 (P1): now also U2.~ (VMOT)
- net at P6.2 (P2): now also U2.~ (VMOT)
- net at P6.3 (P3): now also U2.~ (VMOT)
- net at P6.4 (P4): now also U2.~ (VMOT)
- net at P7.1 (P1): now also U3.~ (VMOT)
- net at P7.2 (P2): now also U3.~ (VMOT)
- net at P7.3 (P3): now also U3.~ (VMOT)
- net at P7.4 (P4): now also U3.~ (VMOT)
- net at P8.1 (P1): now also U4.~ (VMOT)
- net at P8.2 (P2): now also U4.~ (VMOT)
- net at P8.3 (P3): now also U4.~ (VMOT)
- net at P8.4 (P4): now also U4.~ (VMOT)
Other:
- moved on the sheet: P5, P6, P7, P8

Commit message: PCB
Parts:
- C1, C2, C3, C4: footprint (none) -> Capacitors_ThroughHole:C_Rect_L7.0mm_W2.5mm_P5.00mm
- P5: value CONN_01X04 -> stepstick1; footprint (none) -> Pin_Headers:Pin_Header_Straight_1x04_Pitch2.54mm
- P6: value CONN_01X04 -> stepstick3; footprint (none) -> Pin_Headers:Pin_Header_Straight_1x04_Pitch2.54mm
- P7: value CONN_01X04 -> stepstick2; footprint (none) -> Pin_Headers:Pin_Header_Straight_1x04_Pitch2.54mm
- P8: value CONN_01X04 -> stepstick4; footprint (none) -> Pin_Headers:Pin_Header_Straight_1x04_Pitch2.54mm
- U1, U2, U3, U4: footprint (none) -> robot_1A:Stepstick
Changed lines of the file:
@@
 $Descr A4 11693 8268
 encoding utf-8
-Sheet 2 8
+Sheet 2 9
 Title ""
 Date ""
@@
 F 0 "U1" H 400 11300 60  0000 C CNN
 F 1 "Stepstick" H 2750 19450 60  0000 C CNN
-F 2 "" H 2750 19550 60  0001 C CNN
+F 2 "robot_1A:Stepstick" H 2750 19550 60  0001 C CNN
 F 3 "" H 2750 19550 60  0001 C CNN
 	1    350  11250
@@
 F 0 "C1" H 3925 3100 50  0000 L CNN
 F 1 "100µ" H 3925 2900 50  0000 L CNN
-F 2 "" H 3938 2850 50  0000 C CNN
+F 2 "Capacitors_ThroughHole:C_Rect_L7.0mm_W2.5mm_P5.00mm" H 3938 2850 50  0001 C CNN
 F 3 "" H 3900 3000 50  0000 C CNN
 	1    3900 3000
@@
 F 0 "U2" H 550 14350 60  0000 C CNN
 F 1 "Stepstick" H 2900 22500 60  0000 C CNN
-F 2 "" H 2900 22600 60  0001 C CNN
+F 2 "robot_1A:Stepstick" H 2900 22600 60  0001 C CNN
 F 3 "" H 2900 22600 60  0001 C CNN
 	1    500  14300
@@
 F 0 "C2" H 4075 6150 50  0000 L CNN
 F 1 "100µ" H 4075 5950 50  0000 L CNN
-F 2 "" H 4088 5900 50  0000 C CNN
+F 2 "Capacitors_ThroughHole:C_Rect_L7.0mm_W2.5mm_P5.00mm" H 4088 5900 50  0001 C CNN
 F 3 "" H 4050 6050 50  0000 C CNN
 	1    4050 6050
@@
 F 0 "U3" H 5600 10450 60  0000 C CNN
 F 1 "Stepstick" H 7950 18600 60  0000 C CNN
-F 2 "" H 7950 18700 60  0001 C CNN
+F 2 "robot_1A:Stepstick" H 7950 18700 60  0001 C CNN
 F 3 "" H 7950 18700 60  0001 C CNN
 	1    5550 10400
@@
 F 0 "C3" H 9125 2250 50  0000 L CNN
 F 1 "100µ" H 9125 2050 50  0000 L CNN
-F 2 "" H 9138 2000 50  0000 C CNN
+F 2 "Capacitors_ThroughHole:C_Rect_L7.0mm_W2.5mm_P5.00mm" H 9138 2000 50  0001 C CNN
 F 3 "" H 9100 2150 50  0000 C CNN
 	1    9100 2150
@@
 F 0 "U4" H 5800 12950 60  0000 C CNN
 F 1 "Stepstick" H 8150 21100 60  0000 C CNN
-F 2 "" H 8150 21200 60  0001 C CNN
+F 2 "robot_1A:Stepstick" H 8150 21200 60  0001 C CNN
 F 3 "" H 8150 21200 60  0001 C CNN
 	1    5750 12900
@@
 F 0 "C4" H 9325 4750 50  0000 L CNN
 F 1 "100µ" H 9325 4550 50  0000 L CNN
-F 2 "" H 9338 4500 50  0000 C CNN
+F 2 "Capacitors_ThroughHole:C_Rect_L7.0mm_W2.5mm_P5.00mm" H 9338 4500 50  0001 C CNN
 F 3 "" H 9300 4650 50  0000 C CNN
 	1    9300 4650
@@
 P 4000 3500
 F 0 "P5" H 4000 3750 50  0000 C CNN
-F 1 "CONN_01X04" V 4100 3500 50  0000 C CNN
-F 2 "" H 4000 3500 50  0000 C CNN
+F 1 "stepstick1" V 4100 3500 50  0000 C CNN
+F 2 "Pin_Headers:Pin_Header_Straight_1x04_Pitch2.54mm" H 4000 3500 50  0001 C CNN
 F 3 "" H 4000 3500 50  0000 C CNN
 	1    4000 3500
@@
 P 4400 6550
 F 0 "P6" H 4400 6800 50  0000 C CNN
-F 1 "CONN_01X04" V 4500 6550 50  0000 C CNN
-F 2 "" H 4400 6550 50  0000 C CNN
+F 1 "stepstick3" V 4500 6550 50  0000 C CNN
+F 2 "Pin_Headers:Pin_Header_Straight_1x04_Pitch2.54mm" H 4400 6550 50  0001 C CNN
 F 3 "" H 4400 6550 50  0000 C CNN
 	1    4400 6550
@@
 P 9300 2650
 F 0 "P7" H 9300 2900 50  0000 C CNN
-F 1 "CONN_01X04" V 9400 2650 50  0000 C CNN
-F 2 "" H 9300 2650 50  0000 C CNN
+F 1 "stepstick2" V 9400 2650 50  0000 C CNN
+F 2 "Pin_Headers:Pin_Header_Straight_1x04_Pitch2.54mm" H 9300 2650 50  0001 C CNN
 F 3 "" H 9300 2650 50  0000 C CNN
 	1    9300 2650
@@
 P 9700 5150
 F 0 "P8" H 9700 5400 50  0000 C CNN
-F 1 "CONN_01X04" V 9800 5150 50  0000 C CNN
-F 2 "" H 9700 5150 50  0000 C CNN
+F 1 "stepstick4" V 9800 5150 50  0000 C CNN
+F 2 "Pin_Headers:Pin_Header_Straight_1x04_Pitch2.54mm" H 9700 5150 50  0001 C CNN
 F 3 "" H 9700 5150 50  0000 C CNN
 	1    9700 5150

Commit message: fin PCB
Parts:
- U1, U2, U3, U4: symbol Stepstick -> Stepstick-RESCUE-carte-asser-1A-2016-2017
- renumbered P5 to P4, P6 to P5, P7 to P6, P8 to P7
Connections:
- net +15V: now also U1.16 (VMOT), U2.16 (VMOT), U3.16 (VMOT), U4.16 (VMOT); no longer U1.~ (VMOT), U2.~ (VMOT), U3.~ (VMOT), U4.~ (VMOT)
- net +5V: now also U1.3 (SLEEP), U1.4 (RESET), U2.3 (SLEEP), U2.4 (RESET), U3.3 (SLEEP), U3.4 (RESET), U4.3 (SLEEP), U4.4 (RESET); no longer U1.~ (VMOT), U2.~ (VMOT), U3.~ (VMOT), U4.~ (VMOT)
- net GND: now also U1.15 (GND), U1.9 (GND), U2.15 (GND), U2.9 (GND), U3.15 (GND), U3.9 (GND), U4.15 (GND), U4.9 (GND); no longer U1.~ (VMOT), U2.~ (VMOT), U3.~ (VMOT), U4.~ (VMOT)
- net dir-p1: now also U1.1 (DIR); no longer U1.~ (VMOT)
- net dir-p2: now also U3.1 (DIR); no longer U3.~ (VMOT)
- net dir-r1: now also U2.1 (DIR); no longer U2.~ (VMOT)
- net dir-r2: now also U4.1 (DIR); no longer U4.~ (VMOT)
- net enable-p1: now also U1.8 (ENABLE); no longer U1.~ (VMOT)
- net enable-p2: now also U3.8 (ENABLE); no longer U3.~ (VMOT)
- net enable-r1: now also U2.8 (ENABLE); no longer U2.~ (VMOT)
- net enable-r2: now also U4.8 (ENABLE); no longer U4.~ (VMOT)
- net pince-M0: now also U1.7 (M0), U3.7 (M0); no longer U1.~ (VMOT), U3.~ (VMOT)
- net pince-M1: now also U1.6 (M1), U3.6 (M1); no longer U1.~ (VMOT), U3.~ (VMOT)
- net pince-M2: now also U1.5 (M2), U3.5 (M2); no longer U1.~ (VMOT), U3.~ (VMOT)
- net roue-M0: now also U2.7 (M0), U4.7 (M0); no longer U2.~ (VMOT), U4.~ (VMOT)
- net roue-M1: now also U2.6 (M1), U4.6 (M1); no longer U2.~ (VMOT), U4.~ (VMOT)
- net roue-M2: now also U2.5 (M2), U4.5 (M2); no longer U2.~ (VMOT), U4.~ (VMOT)
- net step-p1: now also U1.2 (STEP); no longer U1.~ (VMOT)
- net step-p2: now also U3.2 (STEP); no longer U3.~ (VMOT)
- net step-r1: now also U2.2 (STEP); no longer U2.~ (VMOT)
- net step-r2: now also U4.2 (STEP); no longer U4.~ (VMOT)
- net at P4.1 (P1): now also U1.14 (B2); no longer U1.~ (VMOT)
- net at P4.2 (P2): now also U1.13 (B1); no longer U1.~ (VMOT)
- net at P4.3 (P3): now also U1.12 (A2); no longer U1.~ (VMOT)
- net at P4.4 (P4): now also U1.11 (A1); no longer U1.~ (VMOT)
- net at P5.1 (P1): now also U2.14 (B2); no longer U2.~ (VMOT)
- net at P5.2 (P2): now also U2.13 (B1); no longer U2.~ (VMOT)
- net at P5.3 (P3): now also U2.12 (A2); no longer U2.~ (VMOT)
- net at P5.4 (P4): now also U2.11 (A1); no longer U2.~ (VMOT)
- net at P6.1 (P1): now also U3.14 (B2); no longer U3.~ (VMOT)
- net at P6.2 (P2): now also U3.13 (B1); no longer U3.~ (VMOT)
- net at P6.3 (P3): now also U3.12 (A2); no longer U3.~ (VMOT)
- net at P6.4 (P4): now also U3.11 (A1); no longer U3.~ (VMOT)
- net at P7.1 (P1): now also U4.14 (B2); no longer U4.~ (VMOT)
- net at P7.2 (P2): now also U4.13 (B1); no longer U4.~ (VMOT)
- net at P7.3 (P3): now also U4.12 (A2); no longer U4.~ (VMOT)
- net at P7.4 (P4): now also U4.11 (A1); no longer U4.~ (VMOT)
- new net +3V3: U1.10 (FAULT), U3.10 (FAULT)
- new net Carte_Fault_1: U2.10 (FAULT)
- new net Carte_Fault_2: U4.10 (FAULT)
Changed lines of the file:
@@
 EESchema Schematic File Version 2
+LIBS:carte-asser-1A-2016-2017-rescue
 LIBS:power
 LIBS:device
@@
 $Descr A4 11693 8268
 encoding utf-8
-Sheet 2 9
+Sheet 2 10
 Title ""
 Date ""
@@
 $EndDescr
 $Comp
-L Stepstick U1
+L Stepstick-RESCUE-carte-asser-1A-2016-2017 U1
 U 1 1 589208C0
 P 350 11250
@@
 step-p1
 $Comp
-L GND #PWR04
+L GND #PWR02
 U 1 1 58920AD5
 P 3600 4450
-F 0 "#PWR04" H 3600 4200 50  0001 C CNN
+F 0 "#PWR02" H 3600 4200 50  0001 C CNN
 F 1 "GND" H 3600 4300 50  0000 C CNN
 F 2 "" H 3600 4450 50  0000 C CNN
@@
 dir-p1
 $Comp
-L GND #PWR05
+L GND #PWR03
 U 1 1 58920B1E
 P 5150 3400
-F 0 "#PWR05" H 5150 3150 50  0001 C CNN
+F 0 "#PWR03" H 5150 3150 50  0001 C CNN
 F 1 "GND" H 5150 3250 50  0000 C CNN
 F 2 "" H 5150 3400 50  0000 C CNN
@@
 pince-M2
 $Comp
-L Stepstick U2
+L Stepstick-RESCUE-carte-asser-1A-2016-2017 U2
 U 1 1 58932F20
 P 500 14300
@@
 step-r1
 $Comp
-L GND #PWR06
+L GND #PWR04
 U 1 1 58932F2C
 P 3750 7500
-F 0 "#PWR06" H 3750 7250 50  0001 C CNN
+F 0 "#PWR04" H 3750 7250 50  0001 C CNN
 F 1 "GND" H 3750 7350 50  0000 C CNN
 F 2 "" H 3750 7500 50  0000 C CNN
@@
 dir-r1
 $Comp
-L GND #PWR07
+L GND #PWR05
 U 1 1 58932F36
 P 5300 6450
-F 0 "#PWR07" H 5300 6200 50  0001 C CNN
+F 0 "#PWR05" H 5300 6200 50  0001 C CNN
 F 1 "GND" H 5300 6300 50  0000 C CNN
 F 2 "" H 5300 6450 50  0000 C CNN
@@
 roue-M2
 $Comp
-L Stepstick U3
+L Stepstick-RESCUE-carte-asser-1A-2016-2017 U3
 U 1 1 5893342A
 P 5550 10400
@@
 enable-p2
 $Comp
-L GND #PWR08
+L GND #PWR06
 U 1 1 58933435
 P 8800 3600
-F 0 "#PWR08" H 8800 3350 50  0001 C CNN
+F 0 "#PWR06" H 8800 3350 50  0001 C CNN
 F 1 "GND" H 8800 3450 50  0000 C CNN
 F 2 "" H 8800 3600 50  0000 C CNN
@@
 pince-M2
 $Comp
-L GND #PWR09
+L GND #PWR07
 U 1 1 589334BA
 P 10350 2500
-F 0 "#PWR09" H 10350 2250 50  0001 C CNN
+F 0 "#PWR07" H 10350 2250 50  0001 C CNN
 F 1 "GND" H 10350 2350 50  0000 C CNN
 F 2 "" H 10350 2500 50  0000 C CNN
@@
 $EndComp
 $Comp
-L Stepstick U4
+L Stepstick-RESCUE-carte-asser-1A-2016-2017 U4
 U 1 1 58933897
 P 5750 12900
@@
 enable-r2
 $Comp
-L GND #PWR010
+L GND #PWR08
 U 1 1 589338A2
 P 9000 6100
-F 0 "#PWR010" H 9000 5850 50  0001 C CNN
+F 0 "#PWR08" H 9000 5850 50  0001 C CNN
 F 1 "GND" H 9000 5950 50  0000 C CNN
 F 2 "" H 9000 6100 50  0000 C CNN
@@
 roue-M2
 $Comp
-L GND #PWR011
+L GND #PWR09
 U 1 1 589338BF
 P 10550 5000
-F 0 "#PWR011" H 10550 4750 50  0001 C CNN
+F 0 "#PWR09" H 10550 4750 50  0001 C CNN
 F 1 "GND" H 10550 4850 50  0000 C CNN
 F 2 "" H 10550 5000 50  0000 C CNN
@@
 step-r2
 $Comp
-L CONN_01X04 P5
+L CONN_01X04 P4
 U 1 1 5893C81B
 P 4000 3500
-F 0 "P5" H 4000 3750 50  0000 C CNN
+F 0 "P4" H 4000 3750 50  0000 C CNN
 F 1 "stepstick1" V 4100 3500 50  0000 C CNN
 F 2 "Pin_Headers:Pin_Header_Straight_1x04_Pitch2.54mm" H 4000 3500 50  0001 C CNN
@@
 	9850 4500 9850 3650
 $Comp
-L CONN_01X04 P6
+L CONN_01X04 P5
 U 1 1 589CC6B5
 P 4400 6550
-F 0 "P6" H 4400 6800 50  0000 C CNN
+F 0 "P5" H 4400 6800 50  0000 C CNN
 F 1 "stepstick3" V 4500 6550 50  0000 C CNN
 F 2 "Pin_Headers:Pin_Header_Straight_1x04_Pitch2.54mm" H 4400 6550 50  0001 C CNN
@@
 $EndComp
 $Comp
-L CONN_01X04 P7
+L CONN_01X04 P6
 U 1 1 589CC98E
 P 9300 2650
-F 0 "P7" H 9300 2900 50  0000 C CNN
+F 0 "P6" H 9300 2900 50  0000 C CNN
 F 1 "stepstick2" V 9400 2650 50  0000 C CNN
 F 2 "Pin_Headers:Pin_Header_Straight_1x04_Pitch2.54mm" H 9300 2650 50  0001 C CNN
@@
 $EndComp
 $Comp
-L CONN_01X04 P8
+L CONN_01X04 P7
 U 1 1 589CCBB8
 P 9700 5150
-F 0 "P8" H 9700 5400 50  0000 C CNN
+F 0 "P7" H 9700 5400 50  0000 C CNN
 F 1 "stepstick4" V 9800 5150 50  0000 C CNN
 F 2 "Pin_Headers:Pin_Header_Straight_1x04_Pitch2.54mm" H 9700 5150 50  0001 C CNN
@@
 $EndComp
 $Comp
-L +5V #PWR012
+L +5V #PWR010
 U 1 1 589D942D
 P 1000 3750
-F 0 "#PWR012" H 1000 3600 50  0001 C CNN
+F 0 "#PWR010" H 1000 3600 50  0001 C CNN
 F 1 "+5V" H 1000 3890 50  0000 C CNN
 F 2 "" H 1000 3750 50  0000 C CNN
@@
 $EndComp
 $Comp
-L +5V #PWR013
+L +5V #PWR011
 U 1 1 589D9655
 P 1150 6800
-F 0 "#PWR013" H 1150 6650 50  0001 C CNN
+F 0 "#PWR011" H 1150 6650 50  0001 C CNN
 F 1 "+5V" H 1150 6940 50  0000 C CNN
 F 2 "" H 1150 6800 50  0000 C CNN
@@
 $EndComp
 $Comp
-L +15V #PWR014
+L +15V #PWR012
 U 1 1 589D9AAD
 P 4600 4800
-F 0 "#PWR014" H 4600 4650 50  0001 C CNN
+F 0 "#PWR012" H 4600 4650 50  0001 C CNN
 F 1 "+15V" H 4600 4940 50  0000 C CNN
 F 2 "" H 4600 4800 50  0000 C CNN
@@
 $EndComp
 $Comp
-L +15V #PWR015
+L +15V #PWR013
 U 1 1 589D9BD9
 P 4450 1750
-F 0 "#PWR015" H 4450 1600 50  0001 C CNN
+F 0 "#PWR013" H 4450 1600 50  0001 C CNN
 F 1 "+15V" H 4450 1890 50  0000 C CNN
 F 2 "" H 4450 1750 50  0000 C CNN
@@
 $EndComp
 $Comp
-L +15V #PWR016
+L +15V #PWR014
 U 1 1 589D9DAD
 P 9650 1150
-F 0 "#PWR016" H 9650 1000 50  0001 C CNN
+F 0 "#PWR014" H 9650 1000 50  0001 C CNN
 F 1 "+15V" H 9650 1290 50  0000 C CNN
 F 2 "" H 9650 1150 50  0000 C CNN
@@
 $EndComp
 $Comp
-L +15V #PWR017
+L +15V #PWR015
 U 1 1 589DA061
 P 9850 3650
-F 0 "#PWR017" H 9850 3500 50  0001 C CNN
+F 0 "#PWR015" H 9850 3500 50  0001 C CNN
 F 1 "+15V" H 9850 3790 50  0000 C CNN
 F 2 "" H 9850 3650 50  0000 C CNN
@@
 $EndComp
 $Comp
-L +5V #PWR018
+L +5V #PWR016
 U 1 1 589DA411
 P 6200 2900
-F 0 "#PWR018" H 6200 2750 50  0001 C CNN
+F 0 "#PWR016" H 6200 2750 50  0001 C CNN
 F 1 "+5V" H 6200 3040 50  0000 C CNN
 F 2 "" H 6200 2900 50  0000 C CNN
@@
 $EndComp
 $Comp
-L +5V #PWR019
+L +5V #PWR017
 U 1 1 589DA639
 P 6400 5400
-F 0 "#PWR019" H 6400 5250 50  0001 C CNN
+F 0 "#PWR017" H 6400 5250 50  0001 C CNN
 F 1 "+5V" H 6400 5540 50  0000 C CNN
 F 2 "" H 6400 5400 50  0000 C CNN
@@
 Connection ~ 4050 5900
 Connection ~ 4050 6200
+Wire Wire Line
+	3350 4150 4100 4150
+Wire Wire Line
+	4100 4150 4100 4900
+Wire Wire Line
+	8550 3300 9400 3300
+Wire Wire Line
+	9400 3300 9400 4100
+Wire Wire Line
+	4100 4900 2700 4900
+Wire Wire Line
+	9400 4100 8000 4100
+$Comp
+L +3V3 #PWR018
+U 1 1 58C1F8E0
+P 2700 4900
+F 0 "#PWR018" H 2700 4750 50  0001 C CNN
+F 1 "+3V3" H 2700 5040 50  0000 C CNN
+F 2 "" H 2700 4900 50  0000 C CNN
+F 3 "" H 2700 4900 50  0000 C CNN
+	1    2700 4900
+	1    0    0    -1
+$EndComp
+$Comp
+L +3V3 #PWR019
+U 1 1 58C1F90C
+P 8000 4100
+F 0 "#PWR019" H 8000 3950 50  0001 C CNN
+F 1 "+3V3" H 8000 4240 50  0000 C CNN
+F 2 "" H 8000 4100 50  0000 C CNN
+F 3 "" H 8000 4100 50  0000 C CNN
+	1    8000 4100
+	1    0    0    -1
+$EndComp
+Wire Wire Line
+	3500 7200 4500 7200
+Wire Wire Line
+	8750 5800 10000 5800
+Text HLabel 4500 7200 2    60   Input ~ 0
+Carte_Fault_1
+Text HLabel 10000 5800 2    60   Input ~ 0
+Carte_Fault_2
 $EndSCHEMATC
