File: carte-asser-1A-2016-2017/carte-asser-1A-2016-2017.kicad_pcb (KiCad board)
At the start: 2 copper layers, 78 parts, among them P1 led-fusée, P10 dist-capt1, P11 dist-capt4, P12 dist-capt5, P13 dist-capt2, P14 dist-capt3, P15 dist-capt6, P16 cfc4, P17 cfc1, P18 cfc5, P19 cfc2, P2 Balise, P20 cfc3, P21 cfc6, P22 green-captor, P23 blue-captor, P24 alim-color, P25 alim-servo, P26 data-servo, P27 masse-servo, P3 uart-pi, P4 red-captor, P5 stepstick1, P6 stepstick3, P7 stepstick2, P8 stepstick4, P9 cc-motor, U1 Stepstick, U10 LM324, U12 74HC04, U13 74LS126, U2 Stepstick, U3 Stepstick, U4 Stepstick, U5 +5V, U6 MCP1702, U7 +15V, U8 +7.3V, U9 Nucleo-64

Commit message: fin PCB
Parts:
- added R17: R, Discret:R4-LARGE_PADS, F.Cu at (0.00, 0.00)
- added U11: 74HC04, Housings_DIP:DIP-14_W7.62mm, F.Cu at (0.00, 0.00)
- P1: value led-fusée -> Balise
- P10: value dist-capt1 -> cfc1
- P11: value dist-capt4 -> cfc5
- P12: value dist-capt5 -> cfc2
- P13: value dist-capt2 -> cfc3
- P14: value dist-capt3 -> cfc6
- P15: value dist-capt6 -> red-captor
- P16: value cfc4 -> green-captor
- P17: value cfc1 -> blue-captor
- P18: value cfc5 -> alim-color
- P19: value cfc2 -> dist-capt1
- P2: value Balise -> led-fusée
- P20: value cfc3 -> dist-capt4
- P21: value cfc6 -> dist-capt5
- P22: value green-captor -> dist-capt2
- P23: value blue-captor -> dist-capt3
- P24: value alim-color -> dist-capt6
- P4: value red-captor -> stepstick1
- P5: value stepstick1 -> stepstick3
- P6: value stepstick3 -> stepstick2
- P7: value stepstick2 -> stepstick4
- P8: value stepstick4 -> cc-motor
- P9: value cc-motor -> cfc4
- R1: value 300 -> 1k
- R10: value 100M -> 10k
- R12: value 180M -> 100M
- R13: value 1k -> 180M
- R2: value 1.3k -> 300
- R3: value 500 -> 1.3k
- R4: value 10k -> 500
- U10: value LM324 -> Nucleo-64
- U12: value 74HC04 -> 74LS126
- U9: value Nucleo-64 -> LM324
- moved U4 0.70 mm to (257.8, 105.4)
- moved C6 0.40 mm to (17.8, 85.1)
- moved P11 0.40 mm to (185.4, 69.8)
Connections:
- P1 pad 1: Net-(P1-Pad1) -> GND
- P1 pad 2: /command_part/led_fusée -> /command_part/Rx-balise
- P10 pad 2: /command_part/c-distance1 -> /cfc_part/cfc1
- P10 pad 3: GND -> (no net)
- P11 pad 2: /command_part/c-distance4 -> /cfc_part/cfc5
- P11 pad 3: GND -> (no net)
- P12 pad 2: /command_part/c-distance5 -> /cfc_part/cfc2
- P12 pad 3: GND -> (no net)
- P13 pad 2: /command_part/c-distance2 -> /cfc_part/cfc3
- P13 pad 3: GND -> (no net)
- P14 pad 2: /command_part/c-distance3 -> /cfc_part/cfc6
- P14 pad 3: GND -> (no net)
- P15 pad 1: +5V -> Net-(P15-Pad1)
- P15 pad 2: /command_part/c-distance6 -> (no net)
- P15 pad 3: GND -> (no net)
- P16 pad 1: +5V -> Net-(P16-Pad1)
- P16 pad 2: /cfc_part/cfc4 -> (no net)
- P17 pad 1: +5V -> Net-(P17-Pad1)
- P17 pad 2: /cfc_part/cfc1 -> (no net)
- P18 pad 1: +5V -> +8V
- P18 pad 2: /cfc_part/cfc5 -> (no net)
- P19 pad 2: /cfc_part/cfc2 -> /command_part/c-distance1
- P2 pad 1: GND -> Net-(P2-Pad1)
- P2 pad 2: /command_part/Rx-balise -> /command_part/led_fusée
- P2 pad 3: /command_part/Tx-balise -> (no net)
- P2 pad 4: +15V -> (no net)
- P20 pad 2: /cfc_part/cfc3 -> /command_part/c-distance4
- P21 pad 2: /cfc_part/cfc6 -> /command_part/c-distance5
- P22 pad 1: Net-(P22-Pad1) -> +5V
- P23 pad 1: Net-(P23-Pad1) -> +5V
- P24 pad 1: +8V -> +5V
- P8 pad 1: Net-(P8-Pad1) -> Net-(D1-Pad2)
- P8 pad 2: Net-(P8-Pad2) -> Net-(D2-Pad2)
- P8 pad 3: Net-(P8-Pad3) -> (no net)
- P8 pad 4: Net-(P8-Pad4) -> (no net)
- P9 pad 1: Net-(D1-Pad2) -> +5V
- P9 pad 2: Net-(D2-Pad2) -> /cfc_part/cfc4
- R1 pad 1: GND -> Net-(P2-Pad1)
- R1 pad 2: Net-(D6-Pad1) -> GND
- R10 pad 1: Net-(R10-Pad1) -> /cfc_part/cfc6
- R10 pad 2: Net-(P4-Pad1) -> GND
- R11 pad 2: Net-(P22-Pad1) -> Net-(P15-Pad1)
- R12 pad 2: Net-(P23-Pad1) -> Net-(P16-Pad1)
- R13 pad 1: /color_part/c_couleurR -> Net-(R13-Pad1)
- R13 pad 2: Net-(R10-Pad1) -> Net-(P17-Pad1)
- R14 pad 1: /color_part/c_couleurG -> /color_part/c_couleurR
- R15 pad 1: /color_part/c_couleurB -> /color_part/c_couleurG
- R16 pad 1: Net-(P1-Pad1) -> /color_part/c_couleurB
- R16 pad 2: GND -> Net-(R13-Pad1)
- R2 pad 2: Net-(D8-Pad1) -> Net-(D6-Pad1)
- R3 pad 2: Net-(D10-Pad1) -> Net-(D8-Pad1)
- R4 pad 1: /cfc_part/cfc4 -> GND
- R4 pad 2: GND -> Net-(D10-Pad1)
- R5 pad 1: /cfc_part/cfc1 -> /cfc_part/cfc4
- R6 pad 1: /cfc_part/cfc5 -> /cfc_part/cfc1
- R7 pad 1: /cfc_part/cfc2 -> /cfc_part/cfc5
- R8 pad 1: /cfc_part/cfc3 -> /cfc_part/cfc2
- R9 pad 1: /cfc_part/cfc6 -> /cfc_part/cfc3
- U10 pad 1: Net-(R10-Pad1) -> (no net)
- U10 pad 10: +3V3 -> (no net)
- U10 pad 11: GND -> (no net)
- U10 pad 2: Net-(P4-Pad1) -> (no net)
- U10 pad 3: +3V3 -> (no net)
- U10 pad 4: +8V -> (no net)
- U10 pad 5: +3V3 -> (no net)
- U10 pad 6: Net-(P22-Pad1) -> (no net)
- U10 pad 7: Net-(R11-Pad1) -> (no net)
- U10 pad 8: Net-(R12-Pad1) -> (no net)
- U10 pad 9: Net-(P23-Pad1) -> (no net)
- U12 pad 2: Net-(U12-Pad2) -> /command_part/TX-servo
- U12 pad 3: (no net) -> Net-(P26-Pad1)
- U12 pad 4: (no net) -> Net-(U11-Pad2)
- U12 pad 5: (no net) -> Net-(P26-Pad1)
- U12 pad 6: (no net) -> /command_part/RX-servo
- U9 pad 1: (no net) -> Net-(R11-Pad1)
- U9 pad 10: (no net) -> +3V3
- U9 pad 11: (no net) -> GND
- U9 pad 3: (no net) -> +3V3
- U9 pad 4: (no net) -> +8V
- U9 pad 5: (no net) -> +3V3
- U9 pad 6: (no net) -> Net-(P16-Pad1)
- U9 pad 7: (no net) -> Net-(R12-Pad1)
- U9 pad 8: (no net) -> Net-(R13-Pad1)
- U9 pad 9: (no net) -> Net-(P17-Pad1)

Commit message: Commandes
Parts:
- removed C5: 100µ, Capacitors_ThroughHole:C_Rect_L7.0mm_W2.5mm_P5.00mm
- removed C6, C7: 1µ, Capacitors_ThroughHole:C_Rect_L7.0mm_W2.5mm_P5.00mm
- removed U13: 74LS126, Housings_DIP:DIP-14_W7.62mm
- removed U6: MCP1702, TO_SOT_Packages_SMD:SOT89-3_Housing
- added R19: 330, Discret:R4-LARGE_PADS, F.Cu at (142.6, 24.2)
- F1: footprint Discret:R4-LARGE_PADS -> Resistors_SMD:R_2816_HandSoldering
- P1: footprint Pin_Headers:Pin_Header_Straight_1x02_Pitch2.54mm -> Pin_Headers:Pin_Header_Straight_1x04_Pitch2.54mm
- P10, P11, P12, P13, P14: footprint Pin_Headers:Pin_Header_Straight_1x03_Pitch2.54mm -> Pin_Headers:Pin_Header_Straight_1x02_Pitch2.54mm
- P15: footprint Pin_Headers:Pin_Header_Straight_1x03_Pitch2.54mm -> Pin_Headers:Pin_Header_Straight_1x01_Pitch2.54mm
- P16, P17, P18: footprint Pin_Headers:Pin_Header_Straight_1x02_Pitch2.54mm -> Pin_Headers:Pin_Header_Straight_1x01_Pitch2.54mm
- P19, P20, P21: footprint Pin_Headers:Pin_Header_Straight_1x02_Pitch2.54mm -> Pin_Headers:Pin_Header_Straight_1x03_Pitch2.54mm
- P2, P8: footprint Pin_Headers:Pin_Header_Straight_1x04_Pitch2.54mm -> Pin_Headers:Pin_Header_Straight_1x02_Pitch2.54mm
- P22, P23, P24: footprint Pin_Headers:Pin_Header_Straight_1x01_Pitch2.54mm -> Pin_Headers:Pin_Header_Straight_1x03_Pitch2.54mm
- P4: footprint Pin_Headers:Pin_Header_Straight_1x01_Pitch2.54mm -> Pin_Headers:Pin_Header_Straight_1x04_Pitch2.54mm
- R18: value R -> 270
- U10: footprint Housings_DIP:DIP-16_W7.62mm -> robot_1A:Nucleo-64
- U9: footprint robot_1A:Nucleo-64 -> Housings_DIP:DIP-16_W7.62mm
- moved D1 196.2 mm to (110.3, 27.9)
- moved P9 191.8 mm to (87.7, 135.8), turned to 180 degrees
- moved P8 188.3 mm to (101.5, 32.3)
- moved D2 186.7 mm to (110.3, 39.3), turned to 180 degrees
- moved D4 185.8 mm to (110.3, 35.2)
- moved D3 184.2 mm to (110.1, 31.9)
- moved P21 171.5 mm to (40.6, 130.8)
- moved P20 168.6 mm to (40.7, 121.8)
- moved R18 167.5 mm to (137.1, 24.4), turned to 270 degrees
- moved R4 166.9 mm to (64.8, 23.3), turned to 270 degrees
- moved H1 166.1 mm to (119.2, 24.9)
- moved R6 160.1 mm to (58.0, 138.8), turned to 270 degrees
- moved P19 151.8 mm to (40.6, 92.7)
- moved R8 151.2 mm to (66.8, 138.8), turned to 270 degrees
- moved P13 146.4 mm to (80.0, 136.2), turned to 180 degrees
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Connections:
- H1 pad 1: (no net) -> /command_part/enable-cc
- H1 pad 10: (no net) -> Net-(H1-Pad10)
- H1 pad 11: (no net) -> Net-(H1-Pad11)
- H1 pad 12: (no net) -> Net-(H1-Pad12)
- H1 pad 13: (no net) -> Net-(H1-Pad13)
- H1 pad 14: (no net) -> Net-(H1-Pad14)
- H1 pad 15: (no net) -> Net-(H1-Pad15)
- H1 pad 16: (no net) -> Net-(H1-Pad16)
- H1 pad 2: (no net) -> /command_part/speed-cc
- H1 pad 3: (no net) -> Net-(D1-Pad2)
- H1 pad 4: (no net) -> GND
- H1 pad 5: (no net) -> GND
- H1 pad 6: (no net) -> Net-(D2-Pad2)
- H1 pad 7: (no net) -> /command_part/dir-cc
- H1 pad 8: (no net) -> +8V
- H1 pad 9: (no net) -> Net-(H1-Pad9)
- P1 pad 1: GND -> +15V
- P1 pad 2: /command_part/Rx-balise -> Net-(P1-Pad2)
- R18 pad 2: Net-(P26-Pad1) -> +3V3
- U1 pad 1: (no net) -> /command_part/dir-p1
- U1 pad 10: (no net) -> +3V3
- U1 pad 11: (no net) -> Net-(P4-Pad4)
- U1 pad 12: (no net) -> Net-(P4-Pad3)
- U1 pad 13: (no net) -> Net-(P4-Pad2)
- U1 pad 14: (no net) -> Net-(P4-Pad1)
- U1 pad 15: (no net) -> GND
- U1 pad 16: (no net) -> +15V
- U1 pad 2: (no net) -> /command_part/step-p1
- U1 pad 3: (no net) -> +5V
- U1 pad 4: (no net) -> +5V
- U1 pad 5: (no net) -> /command_part/pince-M2
- U1 pad 6: (no net) -> /command_part/pince-M1
- U1 pad 7: (no net) -> /command_part/pince-M0
- U1 pad 8: (no net) -> /command_part/enable-p1
- U1 pad 9: (no net) -> GND
- U10 pad 1: (no net) -> Net-(U10-Pad1)
- U10 pad 10: (no net) -> GND
- U10 pad 11: (no net) -> /command_part/RX-Pi
- U10 pad 12: (no net) -> /command_part/TX-Pi
- U10 pad 13: (no net) -> Net-(U10-Pad13)
- U10 pad 14: (no net) -> Net-(U10-Pad14)
- U10 pad 15: (no net) -> Net-(U10-Pad15)
- U10 pad 16: (no net) -> Net-(U10-Pad16)
- U10 pad 2: (no net) -> /command_part/dir-servo
- U10 pad 3: (no net) -> Net-(U10-Pad3)
- U10 pad 4: (no net) -> /command_part/c-distance6
- U10 pad 5: (no net) -> /command_part/c-distance5
- U10 pad 6: (no net) -> /command_part/c-distance4
- U10 pad 7: (no net) -> /command_part/c-distance3
- U10 pad 8: (no net) -> /command_part/c-distance2
- U10 pad 9: (no net) -> /command_part/c-distance1
- U12 pad 10: (no net) -> +5V
- U12 pad 11: (no net) -> /balise_part/Rx-balise
- U12 pad 12: (no net) -> Net-(P1-Pad3)
- U12 pad 13: (no net) -> +5V
- U12 pad 8: (no net) -> Net-(P1-Pad2)
- U12 pad 9: (no net) -> /balise_part/Tx-balise
- U2 pad 1: (no net) -> /command_part/dir-r1
- U2 pad 10: (no net) -> /command_part/Carte_Fault_1
- U2 pad 11: (no net) -> Net-(P5-Pad4)
- U2 pad 12: (no net) -> Net-(P5-Pad3)
- U2 pad 13: (no net) -> Net-(P5-Pad2)
- U2 pad 14: (no net) -> Net-(P5-Pad1)
- U2 pad 15: (no net) -> GND
- U2 pad 16: (no net) -> +15V
- U2 pad 2: (no net) -> /command_part/step-r1
- U2 pad 3: (no net) -> +5V
- U2 pad 4: (no net) -> +5V
- U2 pad 5: (no net) -> /command_part/roue-M2
- U2 pad 6: (no net) -> /command_part/roue-M1
- U2 pad 7: (no net) -> /command_part/roue-M0
- U2 pad 8: (no net) -> /command_part/enable-r1
- U2 pad 9: (no net) -> GND
- U3 pad 1: (no net) -> /command_part/dir-p2
- U3 pad 10: (no net) -> +3V3
- U3 pad 11: (no net) -> Net-(P6-Pad4)
- U3 pad 12: (no net) -> Net-(P6-Pad3)
- U3 pad 13: (no net) -> Net-(P6-Pad2)
- U3 pad 14: (no net) -> Net-(P6-Pad1)
- U3 pad 15: (no net) -> GND
- U3 pad 16: (no net) -> +15V
- U3 pad 2: (no net) -> /command_part/step-p2
- U3 pad 3: (no net) -> +5V
- U3 pad 4: (no net) -> +5V
- U3 pad 5: (no net) -> /command_part/pince-M2
- U3 pad 6: (no net) -> /command_part/pince-M1
- U3 pad 7: (no net) -> /command_part/pince-M0
- U3 pad 8: (no net) -> /command_part/enable-p2
- U3 pad 9: (no net) -> GND
- U4 pad 1: (no net) -> /command_part/dir-r2
- U4 pad 10: (no net) -> /command_part/Carte_Fault_2
- U4 pad 11: (no net) -> Net-(P7-Pad4)
- U4 pad 12: (no net) -> Net-(P7-Pad3)
- U4 pad 13: (no net) -> Net-(P7-Pad2)
- U4 pad 14: (no net) -> Net-(P7-Pad1)
- U4 pad 15: (no net) -> GND
- U4 pad 16: (no net) -> +15V
- U4 pad 2: (no net) -> /command_part/step-r2
- U4 pad 3: (no net) -> +5V
- U4 pad 4: (no net) -> +5V
- U4 pad 5: (no net) -> /command_part/roue-M2
- U4 pad 6: (no net) -> /command_part/roue-M1
- U4 pad 7: (no net) -> /command_part/roue-M0
- U4 pad 8: (no net) -> /command_part/enable-r2
- U4 pad 9: (no net) -> GND
Routing:
- net GND: track 0.00 -> 737.3 mm
- net +5V: track 0.00 -> 703.8 mm
- net +8V: track 0.00 -> 310.6 mm
- net +15V: track 0.00 -> 300.7 mm
- net +3V3: track 0.00 -> 212.3 mm
- net /color_part/c_couleurR: track 0.00 -> 144.7 mm
- net /command_part/enable-cc: track 0.00 -> 121.0 mm
- net /command_part/pince-M0: track 0.00 -> 110.0 mm
- net /command_part/speed-cc: track 0.00 -> 109.4 mm
- net /command_part/pince-M2: track 0.00 -> 105.1 mm
- net /color_part/c_couleurB: track 0.00 -> 93.7 mm
- net /command_part/dir-servo: track 0.50 -> 88.4 mm
- net /color_part/c_couleurG: track 0.00 -> 81.1 mm
- net /command_part/pince-M1: track 0.00 -> 77.5 mm
- net /command_part/dir-cc: track 0.00 -> 75.8 mm
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- added copper zone on B.Cu, net GND
- added copper zone on F.Cu, net GND
Other:
- net class Default: clearance 0.2 -> 0.254; trace_width 0.25 -> 0.635; via_dia 0.6 -> 1.27; via_drill 0.4 -> 0.381
- rule trace_clearance: 0.2 -> 0.254
- board text added: "+15V"
- board text added: "+5V"
- board text added: "+8V"
- board text added: "Alim servo"
- board text added: "B"
- board text added: "Balise"
- board text added: "Fusée"
- board text added: "G"
- board text added: "GND servo"
- board text added: "Pince 1"
- board text added: "Pince 2"
- board text added: "R"
- board text added: "Robotronik-1A-2016/2017"
- board text added: "Roue 1"
- board text added: "Roue 2"
- board text added: "TX-Pi RX-Pi"
- board text added: "cc motor"
- board text added: "cfc"
- board text added: "dist-capt"
