File: PCB_Robot_sumo_commande/PCB/Robot_sumo.kicad_pcb (KiCad board)
At the start: 2 copper layers, 100 x 100 mm, 64 parts, among them J1 CONN_Batt, J2 CONN_C1, J3 CONN_C3, J4 CONN_C2, J5 CONN_C4, J6 CONN_M1, J7 CONN_M2, J8 CONN_distance, U1 Arduino-nano, U2 LM324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

Commit message: espacement modifié
Routing:
- net GND: track 420.3 -> 405.8 mm
- net +5V: track 382.6 -> 377.3 mm
- net Net-(C1-Pad1): track 46.4 -> 49.7 mm, vias 0 -> 2
Other:
- net class Default: clearance 0.254 -> 0.31
- rule trace_clearance: 0.254 -> 0.31

Commit message: back logo
Parts:
- added G***: LOGO, logo:phelma-logo-exp2, B.Cu at (136.5, 118.7)
