File: Robot_sumo-2017/PCB/R-IR.sch (KiCad schematic (older format))
At the start: 37 parts, among them J2 CONN_C1, J3 CONN_C3, J4 CONN_C2, J5 CONN_C4, U2 LM324

Commit message: components values
Parts:
- C1: value C -> 1nC
- C3: value C -> 100nC
- R2, R3: value R -> 300kR
- R6: value R -> 22kR
- Rlim1: value R -> 82R
- Rmes1: value R -> 10kR
Other:
- note added: "constante de temps=22ms"
- note added: "fc basse= 100Hz"
Changed lines of the file:
@@
 LIBS:arduino-nano
 LIBS:l293
-LIBS:trou-3
 LIBS:Robot_sumo-cache
 EELAYER 25 0
@@
 P 4850 2750
 F 0 "R6" V 4930 2750 50  0000 C CNN
-F 1 "R" V 4850 2750 50  0000 C CNN
+F 1 "22kR" V 4850 2750 50  0000 C CNN
 F 2 "Discret:R4-LARGE_PADS" V 4780 2750 50  0001 C CNN
 F 3 "" H 4850 2750 50  0001 C CNN
@@
 P 5200 2750
 F 0 "C3" H 5225 2850 50  0000 L CNN
-F 1 "C" H 5225 2650 50  0000 L CNN
+F 1 "100nC" H 5225 2650 50  0000 L CNN
 F 2 "Capacitors_THT:C_Rect_L7.0mm_W2.5mm_P5.00mm" H 5238 2600 50  0001 C CNN
 F 3 "" H 5200 2750 50  0001 C CNN
@@
 P 1050 1800
 F 0 "Rlim1" V 1130 1800 50  0000 C CNN
-F 1 "R" V 1050 1800 50  0000 C CNN
+F 1 "82R" V 1050 1800 50  0000 C CNN
 F 2 "Discret:R4-LARGE_PADS" V 980 1800 50  0001 C CNN
 F 3 "" H 1050 1800 50  0001 C CNN
@@
 P 1250 2100
 F 0 "Rmes1" V 1330 2100 50  0000 C CNN
-F 1 "R" V 1250 2100 50  0000 C CNN
+F 1 "10kR" V 1250 2100 50  0000 C CNN
 F 2 "Discret:R4-LARGE_PADS" V 1180 2100 50  0001 C CNN
 F 3 "" H 1250 2100 50  0001 C CNN
@@
 P 2300 2150
 F 0 "R2" V 2380 2150 50  0000 C CNN
-F 1 "R" V 2300 2150 50  0000 C CNN
+F 1 "300kR" V 2300 2150 50  0000 C CNN
 F 2 "Discret:R4-LARGE_PADS" V 2230 2150 50  0001 C CNN
 F 3 "" H 2300 2150 50  0001 C CNN
@@
 P 2300 2550
 F 0 "R3" V 2380 2550 50  0000 C CNN
-F 1 "R" V 2300 2550 50  0000 C CNN
+F 1 "300kR" V 2300 2550 50  0000 C CNN
 F 2 "Discret:R4-LARGE_PADS" V 2230 2550 50  0001 C CNN
 F 3 "" H 2300 2550 50  0001 C CNN
@@
 P 1900 2350
 F 0 "C1" H 1925 2450 50  0000 L CNN
-F 1 "C" H 1925 2250 50  0000 L CNN
+F 1 "1nC" H 1925 2250 50  0000 L CNN
 F 2 "Capacitors_THT:C_Rect_L7.0mm_W2.5mm_P5.00mm" H 1938 2200 50  0001 C CNN
 F 3 "" H 1900 2350 50  0001 C CNN
@@
 	10200 6000 10200 5250
 Connection ~ 10200 5250
+Text Notes 1550 3200 0    60   ~ 0
+fc basse= 100Hz
+Text Notes 4650 2150 0    60   ~ 0
+constante de temps=22ms
 $EndSCHEMATC
