File: Robot_sumo-2017/PCB/Robot_sumo.kicad_pcb (KiCad board)
At the start: 2 copper layers, 70 x 90 mm, 63 parts, among them J1 CONN_Batt, J2 CONN_C1, J3 CONN_C3, J4 CONN_C2, J5 CONN_C4, J6 CONN_M1, J7 CONN_M2, J8 CONN_distance, U1 Arduino-nano, U2 LM324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

Commit message: components values
Other:
- board text added: "PCB_Initiation_1A_v1.0"
Changed lines of the file:
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@@
-(kicad_pcb (version 4) (host pcbnew 4.0.6-e0-6349~53~ubuntu16.04.1)
+(kicad_pcb (version 4) (host pcbnew 4.0.7-e1-6374~58~ubuntu16.04.1)
   (general
     (links 128)
@@
     (area 104.924999 89.855 175.595 180.075001)
     (thickness 1.6)
-    (drawings 5)
+    (drawings 6)
     (tracks 654)
     (zones 0)
@@
   (page A4)
   (layers
-    (0 F.Cu signal hide)
+    (0 F.Cu signal)
     (31 B.Cu signal)
-    (32 B.Adhes user hide)
-    (33 F.Adhes user hide)
+    (32 B.Adhes user)
+    (33 F.Adhes user)
     (34 B.Paste user)
-    (35 F.Paste user hide)
-    (36 B.SilkS user hide)
+    (35 F.Paste user)
+    (36 B.SilkS user)
     (37 F.SilkS user)
     (38 B.Mask user)
@@
     (visible_elements FFFFFF7F)
     (pcbplotparams
-      (layerselection 0x00030_80000001)
-      (usegerberextensions false)
+      (layerselection 0x011fc_80000001)
+      (usegerberextensions true)
       (excludeedgelayer true)
-      (linewidth 0.050000)
+      (linewidth 0.100000)
       (plotframeref false)
       (viasonmask false)
@@
       (psa4output false)
       (plotreference true)
-      (plotvalue true)
+      (plotvalue false)
       (plotinvisibletext false)
       (padsonsilk false)
@@
       (outputformat 1)
       (mirror false)
-      (drillshape 1)
+      (drillshape 0)
       (scaleselection 1)
-      (outputdirectory ""))
+      (outputdirectory ../../../../../export_commande/))
   )
   (net 0 "")
@@
       (xy 0.77232 -3.319656) (xy 0.909639 -3.431017) (xy 0.933808 -3.402492)) (layer F.SilkS) (width 0.01))
   )
+  (gr_text PCB_Initiation_1A_v1.0 (at 125.65 177.77) (layer F.SilkS)
+    (effects (font (size 1.5 1.5) (thickness 0.3)))
+  )
   (gr_text "Robotronik\n" (at 109.35 138.81 90) (layer F.SilkS)
