File: Robot_sumo-2017/PCB/T-IR.sch (KiCad schematic (older format))
At the start: 5 parts, among them U3 NE555

Commit message: components values
Parts:
- C9: value 10nC -> 1nC
- R14: value 60kR -> 68kR
Other:
- note added: "fosc=4,7kHz\n\ncourant max 200mA"
Changed lines of the file:
@@
 LIBS:arduino-nano
 LIBS:l293
-LIBS:trou-3
 LIBS:Robot_sumo-cache
 EELAYER 25 0
@@
 P 6550 2300
 F 0 "R14" V 6630 2300 50  0000 C CNN
-F 1 "60kR" V 6550 2300 50  0000 C CNN
+F 1 "68kR" V 6550 2300 50  0000 C CNN
 F 2 "Discret:R4-LARGE_PADS" V 6480 2300 50  0001 C CNN
 F 3 "" H 6550 2300 50  0001 C CNN
@@
 P 4450 2750
 F 0 "C9" H 4475 2850 50  0000 L CNN
-F 1 "10nC" H 4475 2650 50  0000 L CNN
+F 1 "1nC" H 4475 2650 50  0000 L CNN
 F 2 "Capacitors_THT:C_Rect_L7.0mm_W2.5mm_P5.00mm" H 4488 2600 50  0001 C CNN
 F 3 "" H 4450 2750 50  0001 C CNN
@@
 Wire Wire Line
 	6250 1650 6550 1650
+Text Notes 6750 2600 0    60   ~ 0
+fosc=4,7kHz\n\ncourant max 200mA
 $EndSCHEMATC
