File: Robot_sumo-2017/PCB/uC-part.sch (KiCad schematic (older format))
At the start: 3 parts, among them U1 Arduino-nano

Commit message: last version I hope
Parts:
- added U5, U6, U7: trou-3, Arduino-nano:Trou-3, symbol trou-3
Connections:
- net Echo: now also U1.29 (D11); no longer U1.30 (D12)
- net Trig: now also U1.30 (D12); no longer U1.29 (D11)
Changed lines of the file:
@@
 LIBS:arduino-nano
 LIBS:l293
+LIBS:trou-3
 LIBS:Robot_sumo-cache
 EELAYER 25 0
@@
 NoConn ~ 4100 2700
 Text HLabel 6800 2300 2    60   Input ~ 0
+Trig
+Text HLabel 6800 2500 2    60   Input ~ 0
 Echo
-Text HLabel 6800 2500 2    60   Input ~ 0
-Trig
 Wire Wire Line
 	6550 2300 6800 2300
@@
 NoConn ~ 6550 3300
 NoConn ~ 6550 3500
+$Comp
+L trou-3 U5
+U 1 1 59580D66
+P 4800 1050
+F 0 "U5" H 4800 1050 60  0000 C CNN
+F 1 "trou-3" H 4800 1200 60  0000 C CNN
+F 2 "Arduino-nano:Trou-3" H 4800 1050 60  0001 C CNN
+F 3 "" H 4800 1050 60  0001 C CNN
+	1    4800 1050
+	1    0    0    -1
+$EndComp
+$Comp
+L trou-3 U6
+U 1 1 59580E81
+P 6000 1000
+F 0 "U6" H 6000 1000 60  0000 C CNN
+F 1 "trou-3" H 6000 1150 60  0000 C CNN
+F 2 "Arduino-nano:Trou-3" H 6000 1000 60  0001 C CNN
+F 3 "" H 6000 1000 60  0001 C CNN
+	1    6000 1000
+	1    0    0    -1
+$EndComp
+$Comp
+L trou-3 U7
+U 1 1 59580ED4
+P 6950 1000
+F 0 "U7" H 6950 1000 60  0000 C CNN
+F 1 "trou-3" H 6950 1150 60  0000 C CNN
+F 2 "Arduino-nano:Trou-3" H 6950 1000 60  0001 C CNN
+F 3 "" H 6950 1000 60  0001 C CNN
+	1    6950 1000
+	1    0    0    -1
+$EndComp
 $EndSCHEMATC

Commit message: components values
Parts:
- D1: value LED -> LED_red
- R1: value R -> 500R
Connections:
- no-connect marks 15 -> 18
Changed lines of the file:
@@
 LIBS:arduino-nano
 LIBS:l293
-LIBS:trou-3
 LIBS:Robot_sumo-cache
 EELAYER 25 0
@@
 P 3300 2300
 F 0 "D1" H 3300 2400 50  0000 C CNN
-F 1 "LED" H 3300 2200 50  0000 C CNN
+F 1 "LED_red" H 3300 2200 50  0000 C CNN
 F 2 "LEDs:LED_D5.0mm" H 3300 2300 50  0001 C CNN
 F 3 "" H 3300 2300 50  0001 C CNN
@@
 P 3750 2300
 F 0 "R1" V 3830 2300 50  0000 C CNN
-F 1 "R" V 3750 2300 50  0000 C CNN
+F 1 "500R" V 3750 2300 50  0000 C CNN
 F 2 "Discret:R4-LARGE_PADS" V 3680 2300 50  0001 C CNN
 F 3 "" H 3750 2300 50  0001 C CNN
@@
 	1    0    0    -1
 $EndComp
+NoConn ~ 5250 1050
+NoConn ~ 6450 1000
+NoConn ~ 7400 1000
 $EndSCHEMATC
