File: commande_moteurs_brushless/encodeurs.sch (KiCad schematic (older format))
At the start: 0 parts

Commit message: update
Parts:
- added U? (x2): Encodeur, symbol Encodeur
Connections:
- new net +5V: U?.+5V (1), U?.+5V (1)
- new net Ch_A1: U?.Ch_A (2)
- new net Ch_A2: U?.Ch_A (2)
- new net Ch_B1: U?.Ch_B (4)
- new net Ch_B2: U?.Ch_B (4)
- new net GND: U?.GND (3), U?.GND (3)
Changed lines of the file:
@@
 Comment4 ""
 $EndDescr
+$Comp
+L Encodeur U?
+U 1 1 596AA862
+P 5250 2400
+F 0 "U?" H 5300 2500 60  0000 C CNN
+F 1 "Encodeur" H 5300 2600 60  0000 C CNN
+F 2 "" H 5250 2400 60  0001 C CNN
+F 3 "" H 5250 2400 60  0001 C CNN
+	1    5250 2400
+	1    0    0    -1
+$EndComp
+$Comp
+L Encodeur U?
+U 1 1 596AA88D
+P 5250 3500
+F 0 "U?" H 5300 3600 60  0000 C CNN
+F 1 "Encodeur" H 5300 3700 60  0000 C CNN
+F 2 "" H 5250 3500 60  0001 C CNN
+F 3 "" H 5250 3500 60  0001 C CNN
+	1    5250 3500
+	1    0    0    -1
+$EndComp
+$Comp
+L +5V #PWR?
+U 1 1 596AAF98
+P 4650 2050
+F 0 "#PWR?" H 4650 1900 50  0001 C CNN
+F 1 "+5V" H 4650 2190 50  0000 C CNN
+F 2 "" H 4650 2050 50  0001 C CNN
+F 3 "" H 4650 2050 50  0001 C CNN
+	1    4650 2050
+	1    0    0    -1
+$EndComp
+$Comp
+L +5V #PWR?
+U 1 1 596AAFB0
+P 4650 3150
+F 0 "#PWR?" H 4650 3000 50  0001 C CNN
+F 1 "+5V" H 4650 3290 50  0000 C CNN
+F 2 "" H 4650 3150 50  0001 C CNN
+F 3 "" H 4650 3150 50  0001 C CNN
+	1    4650 3150
+	1    0    0    -1
+$EndComp
+$Comp
+L GND #PWR?
+U 1 1 596AB08B
+P 4500 2400
+F 0 "#PWR?" H 4500 2150 50  0001 C CNN
+F 1 "GND" H 4500 2250 50  0000 C CNN
+F 2 "" H 4500 2400 50  0001 C CNN
+F 3 "" H 4500 2400 50  0001 C CNN
+	1    4500 2400
+	0    1    1    0
+$EndComp
+$Comp
+L GND #PWR?
+U 1 1 596AB0FD
+P 4500 3500
+F 0 "#PWR?" H 4500 3250 50  0001 C CNN
+F 1 "GND" H 4500 3350 50  0000 C CNN
+F 2 "" H 4500 3500 50  0001 C CNN
+F 3 "" H 4500 3500 50  0001 C CNN
+	1    4500 3500
+	0    1    1    0
+$EndComp
+Text HLabel 4500 2250 0    60   Input ~ 0
+Ch_A1
+Text HLabel 4500 2550 0    60   Input ~ 0
+Ch_B1
+Text HLabel 4500 3350 0    60   Input ~ 0
+Ch_A2
+Text HLabel 4500 3650 0    60   Input ~ 0
+Ch_B2
+Wire Wire Line
+	4650 2050 4650 2100
+Wire Wire Line
+	4650 2100 4750 2100
+Wire Wire Line
+	4500 2250 4750 2250
+Wire Wire Line
+	4500 2400 4750 2400
+Wire Wire Line
+	4500 2550 4750 2550
+Wire Wire Line
+	4650 3150 4650 3200
+Wire Wire Line
+	4650 3200 4750 3200
+Wire Wire Line
+	4500 3350 4750 3350
+Wire Wire Line
+	4500 3500 4750 3500
+Wire Wire Line
+	4500 3650 4750 3650
 $EndSCHEMATC

Commit message: footprints
Parts:
- U7, U8: renamed from U?; footprint (none) -> Connectors_Molex:Molex_KK-6410-04_04x2.54mm_Straight
Changed lines of the file:
@@
 $EndDescr
 $Comp
-L Encodeur U?
+L Encodeur U7
 U 1 1 596AA862
 P 5250 2400
-F 0 "U?" H 5300 2500 60  0000 C CNN
+F 0 "U7" H 5300 2500 60  0000 C CNN
 F 1 "Encodeur" H 5300 2600 60  0000 C CNN
-F 2 "" H 5250 2400 60  0001 C CNN
+F 2 "Connectors_Molex:Molex_KK-6410-04_04x2.54mm_Straight" H 5250 2400 60  0001 C CNN
 F 3 "" H 5250 2400 60  0001 C CNN
 	1    5250 2400
@@
 $EndComp
 $Comp
-L Encodeur U?
+L Encodeur U8
 U 1 1 596AA88D
 P 5250 3500
-F 0 "U?" H 5300 3600 60  0000 C CNN
+F 0 "U8" H 5300 3600 60  0000 C CNN
 F 1 "Encodeur" H 5300 3700 60  0000 C CNN
-F 2 "" H 5250 3500 60  0001 C CNN
+F 2 "Connectors_Molex:Molex_KK-6410-04_04x2.54mm_Straight" H 5250 3500 60  0001 C CNN
 F 3 "" H 5250 3500 60  0001 C CNN
 	1    5250 3500
@@
 $EndComp
 $Comp
-L +5V #PWR?
+L +5V #PWR056
 U 1 1 596AAF98
 P 4650 2050
-F 0 "#PWR?" H 4650 1900 50  0001 C CNN
+F 0 "#PWR056" H 4650 1900 50  0001 C CNN
 F 1 "+5V" H 4650 2190 50  0000 C CNN
 F 2 "" H 4650 2050 50  0001 C CNN
@@
 $EndComp
 $Comp
-L +5V #PWR?
+L +5V #PWR057
 U 1 1 596AAFB0
 P 4650 3150
-F 0 "#PWR?" H 4650 3000 50  0001 C CNN
+F 0 "#PWR057" H 4650 3000 50  0001 C CNN
 F 1 "+5V" H 4650 3290 50  0000 C CNN
 F 2 "" H 4650 3150 50  0001 C CNN
@@
 $EndComp
 $Comp
-L GND #PWR?
+L GND #PWR058
 U 1 1 596AB08B
 P 4500 2400
-F 0 "#PWR?" H 4500 2150 50  0001 C CNN
+F 0 "#PWR058" H 4500 2150 50  0001 C CNN
 F 1 "GND" H 4500 2250 50  0000 C CNN
 F 2 "" H 4500 2400 50  0001 C CNN
@@
 $EndComp
 $Comp
-L GND #PWR?
+L GND #PWR059
 U 1 1 596AB0FD
 P 4500 3500
-F 0 "#PWR?" H 4500 3250 50  0001 C CNN
+F 0 "#PWR059" H 4500 3250 50  0001 C CNN
 F 1 "GND" H 4500 3350 50  0000 C CNN
 F 2 "" H 4500 3500 50  0001 C CNN
