File: commande_moteurs_brushless/motor_part.sch (KiCad schematic (older format))
At the start: 18 parts

Commit message: update
Parts:
- added C?: C, symbol C
- added Cboot?: 220nC, symbol C
- added Cen?: 5,6nC, symbol C
- added Coff?: 1nC, symbol C
- added Cp?, Cpul?: 10nC, symbol C
- added D? (x2): 1N4148, symbol D_ALT
- added K?: Maxon-200142, symbol Maxon-200142
- added R? (x2): R, symbol R
- added Rdd?: 1kR, symbol R
- added Ren?: 100kR, symbol R
- added Roff?: 33kR, symbol R
- added Rp?: 100R, symbol R
- added Rpul?: 47kR, symbol R
- added Rsense?: 0.03R, symbol R
- added U?: L6235D, symbol L6235D
Connections:
- net +3V3: now also R?.2, Rdd?.2
- net +5V: now also K?.11 (V_Hall)
- net GND: now also C?.2, Cen?.2, Coff?.2, Cpul?.2, K?.7 (GND), R?.1, Roff?.2, Rpul?.2, Rsense?.2, U?.18 (GND), U?.19 (GND), U?.6 (GND), U?.7 (GND)
- net VCC: now also Cboot?.2, D?.2 (A), U?.17 (VS_B), U?.20 (VS_A)
- net Vref: now also C?.1, R?.1, R?.2, U?.13 (VREF)
- new net: K?.9 (Hall_sensor_1), U?.1 (H1)
- new net: Rsense?.1, U?.10 (SENSE_B), U?.3 (SENSE_A)
- new net: K?.5 (Motor_winding_3), K?.6 (Motor_winding_3), U?.16 (OUT_3)
- new net: K?.3 (Motor_winding_2), K?.4 (Motor_winding_2), U?.21 (OUT_2)
- new net: K?.8 (Hall_sensor_2), U?.23 (H2)
- new net: K?.10 (Hall_sensor_3), U?.24 (H3)
- new net: K?.1 (Motor_winding_1), K?.2 (Motor_winding_1), U?.5 (OUT_1)
- new net: D?.1 (K), D?.2 (A), Rp?.2
- new net: Cp?.2, Rp?.1
- new net BRAKE_2: U?.14 (BRAKE)
- new net DIAG_2: Cen?.1, Ren?.1, U?.12 (EN), U?.2 (DIAG)
- new net DIR_2: U?.11 (FWD/REV)
- new net EN_2: Ren?.2
- new net RCOFF2: Coff?.1, Roff?.1, U?.4 (RCOFF)
- new net RCPULSE2: Cpul?.1, Rpul?.1, U?.9 (RCPULSE)
- new net TACHO_2: Rdd?.1, U?.8 (TACHO)
- new net VBOOT2: Cboot?.1, D?.1 (K), U?.15 (VBOOT)
- new net VCP2: Cp?.1, U?.22 (VCP)
Other:
- moved on the sheet: C?, Cboot?, Cen?, Coff?, Cp?, Cpul?, D?, K?, R?, Rdd?, Ren?, Roff?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

Commit message: footprints
Parts:
- C1, C2: renamed from C?; footprint (none) -> Capacitors_SMD:C_1206_HandSoldering
- Cboot1, Cboot2: renamed from Cboot?; footprint (none) -> Capacitors_SMD:C_1206_HandSoldering
- Cen1, Cen2: renamed from Cen?; footprint (none) -> Capacitors_SMD:C_1206_HandSoldering
- Coff1, Coff2: renamed from Coff?; footprint (none) -> Capacitors_SMD:C_1206_HandSoldering
- Cp1, Cp2: renamed from Cp?; footprint (none) -> Capacitors_SMD:C_1206_HandSoldering
- Cpul1, Cpul2: renamed from Cpul?; footprint (none) -> Capacitors_SMD:C_1206_HandSoldering
- D1, D2, D3, D4: renamed from D?; footprint (none) -> Diodes_SMD:D_SOD-123
- R1, R2, R3, R4: renamed from R?; footprint (none) -> Resistors_SMD:R_1206_HandSoldering
- Rdd1, Rdd2: renamed from Rdd?; footprint (none) -> Resistors_SMD:R_1206_HandSoldering
- Ren1, Ren2: renamed from Ren?; footprint (none) -> Resistors_SMD:R_1206_HandSoldering
- Roff1, Roff2: renamed from Roff?; footprint (none) -> Resistors_SMD:R_1206_HandSoldering
- Rp1, Rp2: renamed from Rp?; footprint (none) -> Resistors_SMD:R_1206_HandSoldering
- Rpul1, Rpul2: renamed from Rpul?; footprint (none) -> Resistors_SMD:R_1206_HandSoldering
- Rsense1, Rsense2: renamed from Rsense?; footprint (none) -> Resistors_THT:R_Axial_DIN0414_L11.9mm_D4.5mm_P20.32mm_Horizontal
- U1, U2: renamed from U?; footprint (none) -> Housings_SOIC:SOIC-24_7.5x15.4mm_Pitch1.27mm
- gave numbers to parts that had none: 2
