File: commande_moteurs_brushless/power_part.sch (KiCad schematic (older format))
At the start: 19 parts

Commit message: update
Parts:
- added J?: FAN, symbol CONN_01X02
Connections:
- net GND: now also J?.2 (P2)
- net VCC: now also J?.1 (P1)
Changed lines of the file:
@@
 	4650 2300 4650 2550
 Connection ~ 4800 2550
+$Comp
+L CONN_01X02 J?
+U 1 1 596A9627
+P 5800 1950
+F 0 "J?" H 5800 2100 50  0000 C CNN
+F 1 "FAN" V 5900 1950 50  0000 C CNN
+F 2 "" H 5800 1950 50  0001 C CNN
+F 3 "" H 5800 1950 50  0001 C CNN
+	1    5800 1950
+	1    0    0    -1
+$EndComp
+$Comp
+L GND #PWR?
+U 1 1 596AA4A9
+P 5500 2050
+F 0 "#PWR?" H 5500 1800 50  0001 C CNN
+F 1 "GND" H 5500 1900 50  0000 C CNN
+F 2 "" H 5500 2050 50  0001 C CNN
+F 3 "" H 5500 2050 50  0001 C CNN
+	1    5500 2050
+	1    0    0    -1
+$EndComp
+$Comp
+L VCC #PWR?
+U 1 1 596AA4E5
+P 5500 1850
+F 0 "#PWR?" H 5500 1700 50  0001 C CNN
+F 1 "VCC" H 5500 2000 50  0000 C CNN
+F 2 "" H 5500 1850 50  0001 C CNN
+F 3 "" H 5500 1850 50  0001 C CNN
+	1    5500 1850
+	1    0    0    -1
+$EndComp
+Wire Wire Line
+	5500 1850 5500 1900
+Wire Wire Line
+	5500 1900 5600 1900
+Wire Wire Line
+	5500 2050 5500 2000
+Wire Wire Line
+	5500 2000 5600 2000
 $EndSCHEMATC

Commit message: footprints
Parts:
- C6, C8, C9: renamed from C?; footprint (none) -> Capacitors_THT:CP_Radial_D8.0mm_P3.50mm
- C7: renamed from C?; footprint (none) -> Capacitors_SMD:C_1206_HandSoldering
- D6: renamed from D?; value D_ALT -> D_10A; footprint (none) -> Diodes_SMD:D_SMC_Handsoldering
- D7, D8, D9: renamed from D?; footprint (none) -> Diodes_SMD:D_SMA-SMB_Universal_Handsoldering
- F1: renamed from F?; footprint (none) -> Fuse_Holders_and_Fuses:Fuseholder5x20_horiz_SemiClosed_Casing10x25mm
- J3: renamed from J?; footprint (none) -> Connectors_Molex:Molex_KK-6410-02_02x2.54mm_Straight
- R10, R11, R12, R13, R7, R8, R9: renamed from R?; footprint (none) -> Resistors_SMD:R_1206_HandSoldering
- U4: renamed from U?; footprint (none) -> B plug:B plug 5mm
- U5, U6: renamed from U?; footprint (none) -> TO_SOT_Packages_THT:TO-220_Horizontal
