File: commande_moteurs_brushless/uC.sch (KiCad schematic (older format))
At the start: 3 parts

Commit message: update
Parts:
- added D?: LED_ALT, symbol LED_ALT
- added J?: CONN_01X02, symbol CONN_01X02
- added JP?: Jumper_NC_Dual, symbol Jumper_NC_Dual
- added R?: R, symbol R
- added R?: 10kR, symbol R
Connections:
- net +3V3: now also JP?.3
- net GND: now also D?.1 (K), JP?.1
- net Ch_A2: now reaches U?.18 (PA8)
- net Ch_B2: now reaches U?.19 (PA9)
- net at U?.22 (PA12): now also R?.1
- net at U?.31 (BOOT0/PB8): now also R?.1
- net Ch_A1: now reaches U?.6 (PA0)
- net Ch_B1: now reaches U?.7 (PA1)
- net TX: now reaches U?.8 (PA2)
- net TX: now also J?.2 (P2)
- net RX: now reaches U?.9 (PA3)
- net RX: now also J?.1 (P1)
- new net: D?.2 (A), R?.2
- new net: JP?.2, R?.2
Changed lines of the file:
@@
 Wire Wire Line
 	6650 3400 6800 3400
+$Comp
+L LED_ALT D?
+U 1 1 596A8942
+P 7900 3650
+F 0 "D?" H 7900 3750 50  0000 C CNN
+F 1 "LED_ALT" H 7900 3550 50  0000 C CNN
+F 2 "" H 7900 3650 50  0001 C CNN
+F 3 "" H 7900 3650 50  0001 C CNN
+	1    7900 3650
+	0    -1   -1   0
+$EndComp
+$Comp
+L R R?
+U 1 1 596A89D5
+P 7900 3150
+F 0 "R?" V 7980 3150 50  0000 C CNN
+F 1 "R" V 7900 3150 50  0000 C CNN
+F 2 "" V 7830 3150 50  0001 C CNN
+F 3 "" H 7900 3150 50  0001 C CNN
+	1    7900 3150
+	1    0    0    -1
+$EndComp
+$Comp
+L GND #PWR?
+U 1 1 596A8A12
+P 7900 4100
+F 0 "#PWR?" H 7900 3850 50  0001 C CNN
+F 1 "GND" H 7900 3950 50  0000 C CNN
+F 2 "" H 7900 4100 50  0001 C CNN
+F 3 "" H 7900 4100 50  0001 C CNN
+	1    7900 4100
+	1    0    0    -1
+$EndComp
+Wire Wire Line
+	7900 3300 7900 3500
+Wire Wire Line
+	7900 3800 7900 4100
+Text HLabel 4700 3200 0    60   Input ~ 0
+Ch_A1
+Text HLabel 4700 3300 0    60   Input ~ 0
+Ch_B1
+Text HLabel 6950 3300 2    60   Input ~ 0
+Ch_A2
+Text HLabel 6950 3200 2    60   Input ~ 0
+Ch_B2
+Wire Wire Line
+	4700 3200 4950 3200
+Wire Wire Line
+	4700 3300 4950 3300
+Wire Wire Line
+	6950 3200 6650 3200
+Wire Wire Line
+	6950 3300 6650 3300
+$Comp
+L CONN_01X02 J?
+U 1 1 5974F8CE
+P 3250 4000
+F 0 "J?" H 3250 4150 50  0000 C CNN
+F 1 "CONN_01X02" V 3350 4000 50  0000 C CNN
+F 2 "" H 3250 4000 50  0001 C CNN
+F 3 "" H 3250 4000 50  0001 C CNN
+	1    3250 4000
+	-1   0    0    1
+$EndComp
+Wire Wire Line
+	4350 3400 4950 3400
+Wire Wire Line
+	5450 4200 5450 3900
+Text Label 4350 3400 0    60   ~ 0
+TX
+Text Label 5450 4200 3    60   ~ 0
+RX
+Wire Wire Line
+	3750 3950 3450 3950
+Wire Wire Line
+	3750 4050 3450 4050
+Text Label 3750 3950 0    60   ~ 0
+TX
+Text Label 3750 4050 0    60   ~ 0
+RX
+Wire Wire Line
+	6650 2900 7900 2900
+Wire Wire Line
+	7900 2900 7900 3000
+$Comp
+L R R?
+U 1 1 5974DF8C
+P 5200 1700
+F 0 "R?" V 5280 1700 50  0000 C CNN
+F 1 "10kR" V 5200 1700 50  0000 C CNN
+F 2 "" V 5130 1700 50  0001 C CNN
+F 3 "" H 5200 1700 50  0001 C CNN
+	1    5200 1700
+	0    1    1    0
+$EndComp
+$Comp
+L Jumper_NC_Dual JP?
+U 1 1 5974E017
+P 4900 1700
+F 0 "JP?" H 4950 1600 50  0000 L CNN
+F 1 "Jumper_NC_Dual" H 4900 1800 50  0000 C BNN
+F 2 "" H 4900 1700 50  0001 C CNN
+F 3 "" H 4900 1700 50  0001 C CNN
+	1    4900 1700
+	0    -1   -1   0
+$EndComp
+$Comp
+L +3.3V #PWR?
+U 1 1 5974E084
+P 4900 1300
+F 0 "#PWR?" H 4900 1150 50  0001 C CNN
+F 1 "+3.3V" H 4900 1440 50  0000 C CNN
+F 2 "" H 4900 1300 50  0001 C CNN
+F 3 "" H 4900 1300 50  0001 C CNN
+	1    4900 1300
+	1    0    0    -1
+$EndComp
+$Comp
+L GND #PWR?
+U 1 1 5974E0A8
+P 4900 2100
+F 0 "#PWR?" H 4900 1850 50  0001 C CNN
+F 1 "GND" H 4900 1950 50  0000 C CNN
+F 2 "" H 4900 2100 50  0001 C CNN
+F 3 "" H 4900 2100 50  0001 C CNN
+	1    4900 2100
+	1    0    0    -1
+$EndComp
+Wire Wire Line
+	4900 1300 4900 1450
+Wire Wire Line
+	4900 1950 4900 2100
+Wire Wire Line
+	5000 1700 5050 1700
+Wire Wire Line
+	5350 1700 5550 1700
+Wire Wire Line
+	5550 1700 5550 2200
 $EndSCHEMATC

Commit message: footprints
Parts:
- added C3, C4: 10nC, Capacitors_SMD:C_1206_HandSoldering, symbol C
- added P1: CONN_I2C, Connectors_Molex:Molex_KK-6410-02_02x2.54mm_Straight, symbol CONN_01X02
- added P2: CONN_FREE, Connectors_Molex:Molex_KK-6410-02_02x2.54mm_Straight, symbol CONN_01X02
- added R14: R, Resistors_SMD:R_1206_HandSoldering, symbol R
- added Y1: Crystal_8MHz, Crystals:Crystal_HC49-4H_Vertical, symbol Crystal
- C5: renamed from C?; footprint (none) -> Capacitors_SMD:C_1206_HandSoldering
- D5: renamed from D?; footprint (none) -> Diodes_SMD:D_SMA-SMB_Universal_Handsoldering
- J1: renamed from J?; value CONN_01X02 -> CONN_SERIAL; footprint (none) -> Connectors_Molex:Molex_KK-6410-02_02x2.54mm_Straight
- J2: renamed from J?; footprint (none) -> Connectors_Molex:Molex_KK-6410-04_04x2.54mm_Straight
- JP1: renamed from JP?; footprint (none) -> Pin_Headers:Pin_Header_Straight_1x03_Pitch2.54mm
- R5, R6: renamed from R?; footprint (none) -> Resistors_SMD:R_1206_HandSoldering
- U3: renamed from U?; footprint (none) -> Housings_QFP:LQFP-32_7x7mm_Pitch0.8mm
Connections:
- net GND: now also C3.2, C4.2
- net at U3.10 (PA4): now also P2.2 (P2)
- net at U3.11 (PA5): now also P2.1 (P1)
- net EN_1: now reaches U3.12 (PA6)
- net BRAKE_1: now reaches U3.13 (PA7)
- net DIR_1: now reaches U3.14 (PB0)
- net DIAG_1: now reaches U3.15 (PB1)
- net at U3.2 (PF0): now also C3.1, Y1.1
- net TACHO_1: now reaches U3.20 (PA10)
- net at U3.21 (PA11): now also R6.1
- net TACHO_2: now reaches U3.22 (PA12)
- net TACHO_2: no longer R6.1
- net DIAG_2: now reaches U3.25 (PA15)
- net DIR_2: now reaches U3.26 (PB3)
- net BRAKE_2: now reaches U3.27 (PB4)
- net EN_2: now reaches U3.28 (PB5)
- net I2C_SCL: now reaches U3.29 (PB6)
- net I2C_SCL: now also P1.2 (P2)
- net at U3.3 (PF1): now also R14.1
- net I2C_SDA: now reaches U3.30 (PB7)
- net I2C_SDA: now also P1.1 (P1)
- new net: C4.1, R14.2, Y1.2
Other:
- moved on the sheet: D5, R6
